File: PCB files/motor test board v2/motor test board v2.kicad_pcb (KiCad board)
At the start: 2 copper layers, 78.2 x 49.5 mm, 8 parts, among them J1 Conn_01x02, J2 Conn_01x07, J3 Conn_01x02, U1 MC33887

Commit message: 2/26/2018
Routing:
- net Net-(C2-Pad1): track 84.3 -> 73.9 mm
- net Net-(J1-Pad2): track 47.1 -> 38.5 mm
Changed lines of the file:
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@@
   (general
     (links 19)
-    (no_connects 3)
+    (no_connects 0)
     (area 131.496999 97.206999 209.879001 146.887001)
     (thickness 1.6)
     (drawings 8)
-    (tracks 83)
+    (tracks 74)
     (zones 0)
     (modules 8)
@@
   (segment (start 169.196 103.8703) (end 165.2155 107.8508) (width 0.25) (layer B.Cu) (net 1))
   (segment (start 165.2155 124.841) (end 165.2154 124.841) (width 0.25) (layer B.Cu) (net 1))
-  (segment (start 178.65601 120.55599) (end 178.65601 120.64089) (width 0.25) (layer F.Cu) (net 3))
-  (segment (start 178.65601 120.64089) (end 178.2659 121.031) (width 0.25) (layer F.Cu) (net 3))
-  (segment (start 178.2659 121.031) (end 177.1142 121.031) (width 0.25) (layer F.Cu) (net 3))
-  (segment (start 181.116701 119.619299) (end 180.354701 119.619299) (width 0.25) (layer F.Cu) (net 3))
-  (segment (start 180.354701 119.619299) (end 179.41801 120.55599) (width 0.25) (layer F.Cu) (net 3))
-  (segment (start 179.41801 120.55599) (end 178.65601 120.55599) (width 0.25) (layer F.Cu) (net 3))
-  (segment (start 185.1659 115.5701) (end 181.116701 119.619299) (width 2.64) (layer F.Cu) (net 3))
   (segment (start 190.0664 115.5701) (end 185.1659 115.5701) (width 2.64) (layer F.Cu) (net 3))
   (segment (start 190.0664 115.5701) (end 192.784 118.2877) (width 2.64) (layer F.Cu) (net 3))
@@
   (segment (start 171.4005 136.572) (end 144.526 136.572) (width 2.64) (layer F.Cu) (net 6))
   (segment (start 179.6406 128.3319) (end 171.4005 136.572) (width 2.64) (layer F.Cu) (net 6))
-  (segment (start 179.6406 122.301) (end 179.6406 128.3319) (width 2.64) (layer F.Cu) (net 6))
-  (segment (start 179.6406 122.301) (end 177.1142 122.301) (width 0.5586) (layer F.Cu) (net 6))
   (via (at 165.8484 119.0807) (size 0.6) (layers F.Cu B.Cu) (net 7))
   (segment (start 177.196 107.7331) (end 165.8484 119.0807) (width 0.25) (layer B.Cu) (net 7))
@@
     (connect_pads (clearance 0.508))
     (min_thickness 0.254)
-    (fill yes (arc_segments 16) (thermal_gap 0.508) (thermal_bridge_width 0.508))
+    (fill (arc_segments 16) (thermal_gap 0.508) (thermal_bridge_width 0.508))
     (polygon
       (pts
