File: PCB files/Igniter/_saved_Igniter.sch (KiCad schematic (older format))
At the start: 7 parts

Commit message: 4-2-2018
Connections:
- net labels removed: ->TivaADC
Other:
- note added: "1-5V (SD)\n2-GND (SD)\n3-\n4-Spark plug GND?\n5-Fet Gate\n6-Tiva ADC\n7-GND\n8-5V"
- note removed: "1-5V (SD)\n2-GND (SD)\n3-Tiva A0\n4-Spark plug GND?\n5-Fet Gate\n6-Tiva ADC\n7-GND\n8-5V"
Changed lines of the file:
@@
 $EndComp
 Text Notes 6100 3800 0    60   ~ 0
-1-5V (SD)\n2-GND (SD)\n3-Tiva A0\n4-Spark plug GND?\n5-Fet Gate\n6-Tiva ADC\n7-GND\n8-5V
+1-5V (SD)\n2-GND (SD)\n3-\n4-Spark plug GND?\n5-Fet Gate\n6-Tiva ADC\n7-GND\n8-5V
 Text Notes 3400 4000 0    60   ~ 0
 1-5V\n2-GND\n3-Tiva analog pin
@@
 Text Notes 7675 4375 0    60   ~ 0
 Ground spark plug to neg. terminal of battery?
-Text GLabel 5650 3150 1    60   Input ~ 0
-->TivaADC
 $EndSCHEMATC
