File: PCB files/Igniter/Igniter.sch (KiCad schematic (older format))
At the start: 26 parts, among them J1 SD Header, J2 Battery, J3 PT2, J4 PT1, J5 PT3, J6 PT4, J7 IgnitionCoil, Q1 N MOSFET, SW1 ARM, SW2 Ignite

Commit message: 11/2/2019
-Added board corner standoffs
-More footprint changes
Parts:
- Q1: footprint Package_TO_SOT_THT:TO-220-3_Horizontal_TabDown -> Package_TO_SOT_SMD:TO-263-3_TabPin2
Other:
- note added: "Board Corner Standoffs"
Changed lines of the file:
@@
 F 0 "Q1" H 8991 5686 50  0001 L CNN
 F 1 "N MOSFET" H 8991 5640 50  0000 L CNN
-F 2 "Package_TO_SOT_THT:TO-220-3_Horizontal_TabDown" H 8985 5740 50  0001 C CNN
+F 2 "Package_TO_SOT_SMD:TO-263-3_TabPin2" H 8985 5740 50  0001 C CNN
 F 3 "~" H 8785 5640 50  0001 C CNN
 	1    8785 5640
@@
 L Mechanical:MountingHole MH2
 U 1 1 5DB4BD1A
-P 760 815
-F 0 "MH2" H 860 815 50  0000 L CNN
-F 1 "MountingHole" H 860 770 50  0001 L CNN
-F 2 "MountingHole:MountingHole_2.2mm_M2" H 760 815 50  0001 C CNN
-F 3 "~" H 760 815 50  0001 C CNN
-	1    760  815
+P 3230 805
+F 0 "MH2" H 3330 805 50  0000 L CNN
+F 1 "MountingHole" H 3330 760 50  0001 L CNN
+F 2 "MountingHole:MountingHole_2.2mm_M2" H 3230 805 50  0001 C CNN
+F 3 "~" H 3230 805 50  0001 C CNN
+	1    3230 805
 	1    0    0    -1
 $EndComp
@@
 L Mechanical:MountingHole MH3
 U 1 1 5DB4BE36
-P 755 1735
-F 0 "MH3" H 855 1735 50  0000 L CNN
-F 1 "MountingHole" H 855 1690 50  0001 L CNN
-F 2 "MountingHole:MountingHole_2.2mm_M2" H 755 1735 50  0001 C CNN
-F 3 "~" H 755 1735 50  0001 C CNN
-	1    755  1735
+P 3225 990
+F 0 "MH3" H 3325 990 50  0000 L CNN
+F 1 "MountingHole" H 3325 945 50  0001 L CNN
+F 2 "MountingHole:MountingHole_2.2mm_M2" H 3225 990 50  0001 C CNN
+F 3 "~" H 3225 990 50  0001 C CNN
+	1    3225 990
 	1    0    0    -1
 $EndComp
@@
 L Mechanical:MountingHole MH4
 U 1 1 5DB4BEEA
-P 2015 1740
-F 0 "MH4" H 1915 1740 50  0001 R CNN
-F 1 "MountingHole" H 2115 1695 50  0001 L CNN
-F 2 "MountingHole:MountingHole_2.2mm_M2" H 2015 1740 50  0001 C CNN
-F 3 "~" H 2015 1740 50  0001 C CNN
-	1    2015 1740
+P 3035 990
+F 0 "MH4" H 2935 990 50  0000 R CNN
+F 1 "MountingHole" H 3135 945 50  0001 L CNN
+F 2 "MountingHole:MountingHole_2.2mm_M2" H 3035 990 50  0001 C CNN
+F 3 "~" H 3035 990 50  0001 C CNN
+	1    3035 990
 	1    0    0    1
 $EndComp
@@
 L Mechanical:MountingHole MH1
 U 1 1 5DB4BFCA
-P 2000 810
-F 0 "MH1" V 2000 550 50  0000 L CNN
-F 1 "MountingHole" H 2100 765 50  0001 L CNN
-F 2 "MountingHole:MountingHole_2.2mm_M2" H 2000 810 50  0001 C CNN
-F 3 "~" H 2000 810 50  0001 C CNN
-	1    2000 810
+P 3035 810
+F 0 "MH1" V 3035 550 50  0000 L CNN
+F 1 "MountingHole" H 3135 765 50  0001 L CNN
+F 2 "MountingHole:MountingHole_2.2mm_M2" H 3035 810 50  0001 C CNN
+F 3 "~" H 3035 810 50  0001 C CNN
+	1    3035 810
 	0    1    -1   0
 $EndComp
@@
 Text Notes 8235 5495 0    157  ~ 0
 ?
+Text Notes 2705 680  0    50   ~ 0
+Board Corner Standoffs
 $EndSCHEMATC

Commit message: 11/3/2019
-Added molex footprints for p ducer and solenoid connection
-Completed blade fuse holder footprint
Parts:
- J3, J4, J5, J6: footprint (none) -> Connector_Molex:Molex_Mini-Fit_Jr_5566-04A_2x02_P4.20mm_Vertical
- R1, R2, R3, R4, R5, R6: footprint Resistor_THT:R_Axial_DIN0204_L3.6mm_D1.6mm_P5.08mm_Horizontal -> Resistor_SMD:R_1210_3225Metric_Pad1.42x2.65mm_HandSolder
Changed lines of the file:
@@
 F 0 "J3" H 1367 2915 50  0000 C CNN
 F 1 "PT2" H 1367 3006 50  0000 C CNN
-F 2 "" H 1475 3240 50  0001 C CNN
+F 2 "Connector_Molex:Molex_Mini-Fit_Jr_5566-04A_2x02_P4.20mm_Vertical" H 1475 3240 50  0001 C CNN
 F 3 "~" H 1475 3240 50  0001 C CNN
 	1    1475 3240
@@
 F 0 "J4" H 1132 2920 50  0000 C CNN
 F 1 "PT1" H 1132 3011 50  0000 C CNN
-F 2 "" H 1240 3245 50  0001 C CNN
+F 2 "Connector_Molex:Molex_Mini-Fit_Jr_5566-04A_2x02_P4.20mm_Vertical" H 1240 3245 50  0001 C CNN
 F 3 "~" H 1240 3245 50  0001 C CNN
 	1    1240 3245
@@
 F 0 "J6" H 1402 3535 50  0000 C CNN
 F 1 "PT4" H 1402 3626 50  0000 C CNN
-F 2 "" H 1510 3860 50  0001 C CNN
+F 2 "Connector_Molex:Molex_Mini-Fit_Jr_5566-04A_2x02_P4.20mm_Vertical" H 1510 3860 50  0001 C CNN
 F 3 "~" H 1510 3860 50  0001 C CNN
 	1    1510 3860
@@
 F 0 "J5" H 1137 3535 50  0000 C CNN
 F 1 "PT3" H 1137 3626 50  0000 C CNN
-F 2 "" H 1245 3860 50  0001 C CNN
+F 2 "Connector_Molex:Molex_Mini-Fit_Jr_5566-04A_2x02_P4.20mm_Vertical" H 1245 3860 50  0001 C CNN
 F 3 "~" H 1245 3860 50  0001 C CNN
 	1    1245 3860
@@
 F 0 "R6" V 8463 6140 50  0001 C CNN
 F 1 "10k" V 8555 6140 50  0000 C CNN
-F 2 "Resistor_THT:R_Axial_DIN0204_L3.6mm_D1.6mm_P5.08mm_Horizontal" V 8600 6140 50  0001 C CNN
+F 2 "Resistor_SMD:R_1210_3225Metric_Pad1.42x2.65mm_HandSolder" V 8600 6140 50  0001 C CNN
 F 3 "~" H 8670 6140 50  0001 C CNN
 	1    8670 6140
@@
 F 0 "R5" V 8088 5640 50  0001 C CNN
 F 1 "1k" V 8180 5640 50  0000 C CNN
-F 2 "Resistor_THT:R_Axial_DIN0204_L3.6mm_D1.6mm_P5.08mm_Horizontal" V 8225 5640 50  0001 C CNN
+F 2 "Resistor_SMD:R_1210_3225Metric_Pad1.42x2.65mm_HandSolder" V 8225 5640 50  0001 C CNN
 F 3 "~" H 8295 5640 50  0001 C CNN
 	1    8295 5640
@@
 F 0 "R3" V 8988 2565 50  0001 C CNN
 F 1 "300" V 9080 2565 50  0000 C CNN
-F 2 "Resistor_THT:R_Axial_DIN0204_L3.6mm_D1.6mm_P5.08mm_Horizontal" V 9125 2565 50  0001 C CNN
+F 2 "Resistor_SMD:R_1210_3225Metric_Pad1.42x2.65mm_HandSolder" V 9125 2565 50  0001 C CNN
 F 3 "~" H 9195 2565 50  0001 C CNN
 	1    9195 2565
@@
 F 0 "R4" V 9643 2570 50  0001 C CNN
 F 1 "1200" V 9735 2570 50  0000 C CNN
-F 2 "Resistor_THT:R_Axial_DIN0204_L3.6mm_D1.6mm_P5.08mm_Horizontal" V 9780 2570 50  0001 C CNN
+F 2 "Resistor_SMD:R_1210_3225Metric_Pad1.42x2.65mm_HandSolder" V 9780 2570 50  0001 C CNN
 F 3 "~" H 9850 2570 50  0001 C CNN
 	1    9850 2570
@@
 F 0 "R2" V 3308 2260 50  0001 C CNN
 F 1 "300" V 3510 2260 50  0000 C CNN
-F 2 "Resistor_THT:R_Axial_DIN0204_L3.6mm_D1.6mm_P5.08mm_Horizontal" V 3445 2260 50  0001 C CNN
+F 2 "Resistor_SMD:R_1210_3225Metric_Pad1.42x2.65mm_HandSolder" V 3445 2260 50  0001 C CNN
 F 3 "~" H 3515 2260 50  0001 C CNN
 	1    3515 2260
@@
 F 0 "R1" V 2698 2260 50  0001 C CNN
 F 1 "10k" V 2900 2260 50  0000 C CNN
-F 2 "Resistor_THT:R_Axial_DIN0204_L3.6mm_D1.6mm_P5.08mm_Horizontal" V 2835 2260 50  0001 C CNN
+F 2 "Resistor_SMD:R_1210_3225Metric_Pad1.42x2.65mm_HandSolder" V 2835 2260 50  0001 C CNN
 F 3 "~" H 2905 2260 50  0001 C CNN
 	1    2905 2260

Commit message: 11/3/2019
Added comment
Other:
- note added: "Remove this and do software control"
Changed lines of the file:
@@
 Text Notes 2705 680  0    50   ~ 0
 Board Corner Standoffs
+Text Notes 2385 1850 0    50   ~ 0
+Remove this and do software control
 $EndSCHEMATC

Commit message: 11/7/2019
-Added 7400 series component symbols to kicad
-Begun adding microSD circuit into the board
-Removed physical ignition switch
Parts:
- removed D1: IGNITE-RED, LED_THT:LED_D3.0mm, symbol Device:LED
- removed R1: 10k, Resistor_SMD:R_1210_3225Metric_Pad1.42x2.65mm_HandSolder, symbol Device:R
- removed R2: 300, Resistor_SMD:R_1210_3225Metric_Pad1.42x2.65mm_HandSolder, symbol Device:R
- removed SW2: Ignite, symbol Switch:SW_SPST
- added IC?: 74HC4050, symbol 7400-ic:74HC4050
- added J?: Micro_SD_Card_Det_Hirose_DM3AT, symbol Connector:Micro_SD_Card_Det_Hirose_DM3AT
Connections:
- net labels added: +3V3, CD
- wire segments 47 -> 45
Other:
- note added: "Make unused pins available from the top of shield"
- note removed: "Remove this and do software control"

Commit message: 11/8/2019
-Completed SD card circuit in schematic
-Realized we should regulate 24V to 5V to provide current to stay under the atmega2560 limits
Parts:
- removed IC?: 74HC4050, symbol 7400-ic:74HC4050
- removed J1: SD Header, Connector_PinHeader_2.54mm:PinHeader_1x08_P2.54mm_Vertical, symbol Connector:Conn_01x08_Male
- removed J?: Micro_SD_Card_Det_Hirose_DM3AT, symbol Connector:Micro_SD_Card_Det_Hirose_DM3AT
Connections:
- net labels removed: CD
- wire segments 45 -> 43
- no-connect marks 8 -> 5
Other:
- note added: "Vcc 200mA max current draw\n-Keep total current draw below this value\n-SD card powered by atmega 5V pin\n-Everything else powered by 5V regulator?"
- note added: "approx. 40mA draw"
- note removed: "1 - CD\n2 - CS\n3 - DI\n4 - DO\n5 - CLK\n6 - GND\n7 - 3V\n8 - 5V"
- note removed: "SD breakout board"
- note removed: "actuate solenoids through code\n1 arm switch\n1 ignition switch to trigger code\nIdeal: actuate everything through interface\nIf time does not allow: use analog valve switching\n"

Commit message: 11/8/2019
-Added voltage regulator
-Added 3v3 status led
Parts:
- removed D4: D, Diode_THT:D_DO-15_P12.70mm_Horizontal, symbol Device:D
- removed R5: 1k, Resistor_SMD:R_1210_3225Metric_Pad1.42x2.65mm_HandSolder, symbol Device:R
- added C?: 2.2u, symbol Device:C_Small
- added C?: 1u, symbol Device:C_Small
- added D?: 3V3_GOOD, LED_SMD:LED_1206_3216Metric, symbol Device:LED
- added R?: 200, Resistor_SMD:R_1210_3225Metric_Pad1.42x2.65mm_HandSolder, symbol Device:R
- added U?: MIC5205-5.0, Package_TO_SOT_SMD:SOT-23-5, symbol Regulator_Linear:MIC5205-5.0
- D2, D3: footprint LED_THT:LED_D3.0mm -> LED_SMD:LED_1206_3216Metric
Connections:
- wire segments 43 -> 44
- no-connect marks 5 -> 9
Other:
- note added: "5V regulator"
- note added: "Fix this symbol"
- note added: "Vcc 200mA max current draw\n-Keep total current draw below this value\n-SD card powered by atmega 3V3 pin\n-Everything else powered by 5V regulator"
- note removed: "*"
- note removed: "?"
- note removed: "Vcc 200mA max current draw\n-Keep total current draw below this value\n-SD card powered by atmega 5V pin\n-Everything else powered by 5V regulator?"
- note removed: "approx. 40mA draw"

Commit message: 11/8/2019
-Annotated schematic and generated netlist
-Read netlist to populate PCB
-Schematic is very nearly complete
Parts:
- C1, C2: renamed from C?; footprint (none) -> Capacitor_SMD:C_1206_3216Metric_Pad1.42x1.75mm_HandSolder
- gave numbers to parts that had none: 3
Other:
- moved on the sheet: U1

Commit message: 11/9/2019
-Fixed regulator symbol
-Began adding solenoid valve indicators
Parts:
- removed U1: MIC5205-5.0, Package_TO_SOT_SMD:SOT-23-5, symbol Regulator_Linear:MIC5205-5.0
- added D?: LED, symbol Device:LED
- added R?: 1k2, symbol Device:R
- added U1: MIC3490, Package_TO_SOT_SMD:SOT-23-5_HandSoldering, symbol Regulator_Linear:MIC3490
- R4: value 1200 -> 1k2
Connections:
- net labels added: SOL1, SOL2, SOL3, SOL4, SOL5
- wire segments 44 -> 38
- no-connect marks 9 -> 8
Other:
- note added: "-Board sits at test operator area"
- note added: "-Make unused pins available from the top of shield"
- note added: "NOTES"
- note added: "TBD solenoid indicators"
- note added: "Vcc 200mA max current draw for ATmega2560\n-Keep total current draw below this value\n-SD card powered by atmega 3V3 pin\n-Everything else powered by 5V regulator"
- note removed: "Fix this symbol"
- note removed: "Make unused pins available from the top of shield"
- note removed: "Vcc 200mA max current draw\n-Keep total current draw below this value\n-SD card powered by atmega 3V3 pin\n-Everything else powered by 5V regulator"
