File: PCB files/Igniter/SD.sch (KiCad schematic (older format))
At the start: 2 parts, among them IC1 74HC4050, J1 Micro_SD_Card

Commit message: 11/8/2019
-Added SD circuit footprints
Parts:
- IC1: footprint (none) -> Package_SO:SOP-16_4.4x10.4mm_P1.27mm
- J1: footprint (none) -> Connector_Card:microSD_HC_Hirose_DM3BT-DSF-PEJS
Changed lines of the file:
@@
 F 0 "IC1" H 4115 4602 60  0000 C CNN
 F 1 "74HC4050" H 4115 4496 60  0000 C CNN
-F 2 "" H 4015 3865 60  0001 C CNN
+F 2 "Package_SO:SOP-16_4.4x10.4mm_P1.27mm" H 4015 3865 60  0001 C CNN
 F 3 "" H 4065 3865 60  0001 C CNN
 	1    4115 3865
@@
 F 0 "J1" H 6335 2933 50  0000 C CNN
 F 1 "Micro_SD_Card" H 6335 3024 50  0000 C CNN
-F 2 "" H 7535 4050 50  0001 C CNN
+F 2 "Connector_Card:microSD_HC_Hirose_DM3BT-DSF-PEJS" H 7535 4050 50  0001 C CNN
 F 3 "http://katalog.we-online.de/em/datasheet/693072010801.pdf" H 6385 3750 50  0001 C CNN
 	1    6385 3750

Commit message: 11/8/2019
-Added voltage regulator
-Added 3v3 status led
Connections:
- wire segments 17 -> 15
Other:
- note removed: "10's of mA draw?"
Changed lines of the file:
@@
 L 7400-ic:74HC4050 IC1
 U 1 1 5DC6652F
-P 4115 3865
-F 0 "IC1" H 4115 4602 60  0000 C CNN
-F 1 "74HC4050" H 4115 4496 60  0000 C CNN
-F 2 "Package_SO:SOP-16_4.4x10.4mm_P1.27mm" H 4015 3865 60  0001 C CNN
-F 3 "" H 4065 3865 60  0001 C CNN
-	1    4115 3865
+P 4115 3900
+F 0 "IC1" H 4115 4637 60  0000 C CNN
+F 1 "74HC4050" H 4115 4531 60  0000 C CNN
+F 2 "Package_SO:SOP-16_4.4x10.4mm_P1.27mm" H 4015 3900 60  0001 C CNN
+F 3 "" H 4065 3900 60  0001 C CNN
+	1    4115 3900
 	1    0    0    -1
 $EndComp
@@
 L power:GNDREF #PWR06
 U 1 1 5DC66536
-P 3715 3615
-F 0 "#PWR06" H 3715 3365 50  0001 C CNN
-F 1 "GNDREF" H 3720 3442 50  0001 C CNN
-F 2 "" H 3715 3615 50  0001 C CNN
-F 3 "" H 3715 3615 50  0001 C CNN
-	1    3715 3615
+P 3715 3650
+F 0 "#PWR06" H 3715 3400 50  0001 C CNN
+F 1 "GNDREF" H 3720 3477 50  0001 C CNN
+F 2 "" H 3715 3650 50  0001 C CNN
+F 3 "" H 3715 3650 50  0001 C CNN
+	1    3715 3650
 	1    0    0    -1
 $EndComp
@@
 L power:+3V3 #PWR05
 U 1 1 5DC6653C
-P 3715 3415
-F 0 "#PWR05" H 3715 3265 50  0001 C CNN
-F 1 "+3V3" H 3715 3555 50  0000 C CNN
-F 2 "" H 3715 3415 50  0001 C CNN
-F 3 "" H 3715 3415 50  0001 C CNN
-	1    3715 3415
+P 3715 3450
+F 0 "#PWR05" H 3715 3300 50  0001 C CNN
+F 1 "+3V3" H 3715 3590 50  0000 C CNN
+F 2 "" H 3715 3450 50  0001 C CNN
+F 3 "" H 3715 3450 50  0001 C CNN
+	1    3715 3450
 	1    0    0    -1
 $EndComp
@@
 NoConn ~ 5485 4150
 NoConn ~ 5485 3450
-NoConn ~ 4515 4315
+NoConn ~ 4515 4350
 $Comp
 L power:GNDREF #PWR?
 U 1 1 5DC6A1C2
-P 3715 4315
+P 3715 4350
 AR Path="/5DC6A1C2" Ref="#PWR?"  Part="1"
 AR Path="/5DC64D13/5DC6A1C2" Ref="#PWR09"  Part="1"
-F 0 "#PWR09" H 3715 4065 50  0001 C CNN
-F 1 "GNDREF" H 3720 4142 50  0001 C CNN
-F 2 "" H 3715 4315 50  0001 C CNN
-F 3 "" H 3715 4315 50  0001 C CNN
-	1    3715 4315
+F 0 "#PWR09" H 3715 4100 50  0001 C CNN
+F 1 "GNDREF" H 3720 4177 50  0001 C CNN
+F 2 "" H 3715 4350 50  0001 C CNN
+F 3 "" H 3715 4350 50  0001 C CNN
+	1    3715 4350
 	1    0    0    -1
 $EndComp
 Wire Wire Line
-	4515 4015 4890 4015
-Wire Wire Line
-	4890 4015 4890 3550
+	4515 4050 4890 4050
 Wire Wire Line
 	4890 3550 5485 3550
 Wire Wire Line
-	4515 3815 4750 3815
-Wire Wire Line
-	4515 3915 4945 3915
-Wire Wire Line
-	4945 3915 4945 3650
+	4515 3950 4945 3950
 Wire Wire Line
 	4945 3650 5485 3650
-NoConn ~ 4515 4215
+NoConn ~ 4515 4250
 Wire Wire Line
-	3715 4215 3715 4315
-Connection ~ 3715 4315
+	3715 4250 3715 4350
+Connection ~ 3715 4350
 Wire Wire Line
-	4515 4115 5285 4115
-Text HLabel 3715 3815 0    50   Input ~ 0
+	4515 4150 5285 4150
+Text HLabel 3715 3850 0    50   Input ~ 0
 CLK
-Text HLabel 3715 3915 0    50   Input ~ 0
+Text HLabel 3715 3950 0    50   Input ~ 0
 DI
-Text HLabel 3715 4015 0    50   Input ~ 0
+Text HLabel 3715 4050 0    50   Input ~ 0
 CS
-Text HLabel 3715 4115 0    50   Input ~ 0
+Text HLabel 3715 4150 0    50   Input ~ 0
 DO
-Text Notes 2970 3390 0    50   ~ 0
-10's of mA draw?
 Wire Wire Line
 	5485 3750 5340 3750
@@
 	5340 3950 5340 4390
 Wire Wire Line
-	5285 4115 5285 4050
+	5285 4050 5485 4050
+NoConn ~ 7185 4350
 Wire Wire Line
-	5285 4050 5485 4050
+	4515 3850 5485 3850
 Wire Wire Line
-	5485 3850 4750 3850
+	4945 3650 4945 3950
 Wire Wire Line
-	4750 3850 4750 3815
-NoConn ~ 7185 4350
+	4890 3550 4890 4050
+Wire Wire Line
+	5285 4050 5285 4150
 $EndSCHEMATC

Commit message: 11/12/2019
-Edited fuse holder footprint to have a mechanical hole in the center
-Deleted old, unused IgniterDriver.sch
Parts:
- IC1: symbol 7400-ic:74HC4050 -> Igniter-rescue:74HC4050-7400-ic
- J1: symbol Connector:Micro_SD_Card -> Igniter-rescue:Micro_SD_Card-Connector
Changed lines of the file:
@@
 LIBS:interface
 LIBS:Igniter-cache
-EELAYER 26 0
+EELAYER 29 0
 EELAYER END
 $Descr A4 11693 8268
@@
 $EndComp
 $Comp
-L 7400-ic:74HC4050 IC1
+L Igniter-rescue:74HC4050-7400-ic IC1
 U 1 1 5DC6652F
 P 4115 3900
@@
 $EndComp
 $Comp
-L Connector:Micro_SD_Card J1
+L Igniter-rescue:Micro_SD_Card-Connector J1
 U 1 1 5DC67EC9
 P 6385 3750
