File: PCB files/Pneumatic control/PneuRev1.kicad_pcb (KiCad board)
At the start: 2 copper layers, 154.1 x 77.3 mm, 72 parts, among them J1 SIG_IN, J2 BATT_IN, J3 PNEU, U1 OPA551, U10 OPA551, U11 OPA551, U12 OPA551, U13 OPA551, U2 OPA551, U3 OPA551, U4 OPA551, U5 OPA551, U6 OPA551, U7 OPA551, U8 OPA551, U9 OPA551

Commit message: 2/26/2019
Parts:
- added REF**: MountingHole_4.3mm_M4, Mounting_Holes:MountingHole_4.3mm_M4, F.Cu at (216.6, 65.0)
- added REF**: MountingHole_4.3mm_M4, Mounting_Holes:MountingHole_4.3mm_M4, F.Cu at (69.3, 65.2)
- added REF**: MountingHole_4.3mm_M4, Mounting_Holes:MountingHole_4.3mm_M4, F.Cu at (216.6, 135.4)
- added REF**: MountingHole_4.3mm_M4, Mounting_Holes:MountingHole_4.3mm_M4, F.Cu at (69.4, 135.7)
- moved C13 14.7 mm to (201.3, 68.0)
- moved R35 14.7 mm to (165.1, 81.3)
- moved C12 14.7 mm to (177.2, 67.9)
- moved R29 14.7 mm to (161.3, 74.9)
- moved R32 14.7 mm to (161.3, 72.4)
- moved R38 14.7 mm to (185.4, 74.9)
- moved R39 14.7 mm to (185.4, 72.4)
- moved R40 14.7 mm to (189.2, 81.4)
- moved U10 14.7 mm to (166.2, 67.9)
- moved U13 14.7 mm to (190.3, 68.0)
- moved R20 8.65 mm to (139.3, 74.9)
- moved R23 8.65 mm to (139.4, 72.4)
- moved R26 8.65 mm to (143.1, 81.4)
- moved U7 8.65 mm to (144.2, 68.0)
- moved C9 8.65 mm to (155.3, 68.0)
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Routing:
- net /IN7: track 112.2 -> 131.4 mm
- net /PNU7: track 81.7 -> 92.2 mm
- net /PNU10: track 58.5 -> 68.3 mm
- net /PNU13: track 49.5 -> 56.9 mm, vias 0 -> 4
- net /IN13: track 177.3 -> 184.6 mm
- net Net-(J1-Pad1): track 48.4 -> 43.0 mm
- net /IN10: track 150.5 -> 154.1 mm, vias 2 -> 4
- net Net-(C1-Pad2): track 465.3 -> 462.7 mm, vias 12 -> 28
- net /IN4: track 78.8 -> 80.1 mm, vias 4 -> 5
- net /PNU4: track 106.5 -> 107.7 mm
- net /PNU1: track 133.2 -> 133.3 mm, vias 2 -> 4
Other:
- net class Default: via_drill 0.4 -> 0.3
- rule via_min_drill: 0.3 -> 0.2
- board text added: "+"
- board text added: "-"
- board text added: "IN"
- board text added: "LRDT SPRING 2019 REV 1"
- board text added: "OUT"

Commit message: 12/10/2019
-Selected battery molex connector footprint
-Read netlist
Other:
- outline, holes or cut-outs redrawn
Changed lines of the file:
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@@
-(kicad_pcb (version 4) (host pcbnew 4.0.7)
+(kicad_pcb (version 20171130) (host pcbnew "(5.1.2)-2")
   (general
-    (links 161)
-    (no_connects 53)
-    (area 65.792257 61.697777 219.999783 139.104441)
     (thickness 1.6)
     (drawings 13)
@@
     (zone_45_only no)
     (trace_min 0.2)
-    (segment_width 0.2)
-    (edge_width 0.15)
     (via_size 0.6)
     (via_drill 0.3)
@@
     (uvia_min_size 0.2)
     (uvia_min_drill 0.1)
+    (edge_width 0.15)
+    (segment_width 0.2)
     (pcb_text_width 0.3)
     (pcb_text_size 1.5 1.5)
@@
       (layerselection 0x00030_80000001)
       (usegerberextensions true)
+      (usegerberattributes false)
+      (usegerberadvancedattributes false)
+      (creategerberjobfile false)
       (excludeedgelayer true)
       (linewidth 0.100000)
@@
       (hpglpennumber 1)
       (hpglpenspeed 20)
-      (hpglpendiameter 15)
-      (hpglpenoverlay 2)
+      (hpglpendiameter 15.000000)
       (psnegative false)
       (psa4output false)
@@
       (drillshape 0)
       (scaleselection 1)
-      (outputdirectory ./))
+      (outputdirectory "./"))
   )
   (net 0 "")
@@
     (pad 1 np_thru_hole circle (at 0 0) (size 4.3 4.3) (drill 4.3) (layers *.Cu *.Mask))
   )
+  (gr_line (start 219.923261 64.673484) (end 219.924782 136.033093) (layer Edge.Cuts) (width 0.15))
   (gr_text OUT (at 216.31656 120.45442) (layer F.SilkS)
     (effects (font (size 1.5 1.5) (thickness 0.3)))
@@
     (effects (font (size 1.5 1.5) (thickness 0.3)))
   )
-  (gr_arc (start 216.903013 64.795378) (end 216.928413 61.772778) (angle 88.0744171) (layer Edge.Cuts) (width 0.15))
+  (gr_arc (start 216.903013 64.795378) (end 216.928413 61.772778) (angle 87.20739162) (layer Edge.Cuts) (width 0.15))
   (gr_arc (start 216.902182 136.007693) (end 219.924782 136.033093) (angle 87.91483468) (layer Edge.Cuts) (width 0.15))
-  (gr_arc (start 68.886487 136.011942) (end 68.86956 139.02944) (angle 88.23447828) (layer Edge.Cuts) (width 0.15))
+  (gr_arc (start 68.886487 136.011942) (end 68.87464 139.02944) (angle 88.33092298) (layer Edge.Cuts) (width 0.15))
   (gr_arc (start 68.889858 64.794547) (end 65.867258 64.769147) (angle 88.0744171) (layer Edge.Cuts) (width 0.15))
-  (gr_line (start 68.877138 139.02944) (end 216.98712 139.02944) (layer Edge.Cuts) (width 0.15))
-  (gr_line (start 219.92336 64.72428) (end 219.92476 136.03224) (layer Edge.Cuts) (width 0.15))
+  (gr_line (start 68.87718 139.02944) (end 216.98712 139.02944) (layer Edge.Cuts) (width 0.15))
   (gr_line (start 68.821293 61.7728) (end 216.92616 61.7728) (layer Edge.Cuts) (width 0.15))
   (gr_line (start 65.86982 136.08812) (end 65.86728 64.77254) (layer Edge.Cuts) (width 0.15))
