File: PCB files/TestStandThermo/Thermo/Thermo.sch (KiCad schematic (older format))
At the start: 12 parts

Commit message: Finished thermo schematic
-Taken from adafruit, removed regulator and level shifters
-Created BOM from KiCAD, exported to google drive (Electronics>Solid>BOM)
Parts:
- removed J? (x3): Screw_Terminal_01x02, symbol Connector:Screw_Terminal_01x02
- added C10, C13, C15, C16, C5, C8: 0.1u, Capacitor_SMD:C_0805_2012Metric, symbol Device:C
- added C11, C12, C14, C4, C6, C9: 0.01u, Capacitor_SMD:C_0805_2012Metric, symbol Device:C
- added J2, J5, J6: Screw_Terminal_01x02, TerminalBlock_Phoenix:TerminalBlock_Phoenix_MKDS-1,5-2_1x02_P5.00mm_Horizontal, symbol Connector:Screw_Terminal_01x02
- added J4, J7, J8: Conn_01x08_Female, symbol Connector:Conn_01x08_Female
- added R10, R15, R16, R17, R18, R19, R20, R5, R6, R7, R8, R9: 10k, Resistor_SMD:R_0805_2012Metric, symbol Device:R_US
- added R11, R12, R13, R14, R3, R4: 100, Resistor_SMD:R_0805_2012Metric, symbol Device:R_US
- added U2, U3, U4: MAX31856, Package_SO:TSSOP-14_4.4x5mm_P0.65mm, symbol Sensor_Temperature:MAX31856
- C1, C2, C3, C7: renamed from C?; footprint (none) -> Capacitor_SMD:C_0805_2012Metric
- J1: renamed from J?; footprint (none) -> TerminalBlock_Phoenix:TerminalBlock_Phoenix_MKDS-1,5-2_1x02_P5.00mm_Horizontal
- J3: renamed from J?; value Conn_01x07_Female -> Conn_01x08_Female; symbol Connector:Conn_01x07_Female -> Connector:Conn_01x08_Female
- R1, R2: renamed from R?; footprint (none) -> Resistor_SMD:R_0805_2012Metric
- gave numbers to parts that had none: 1
Connections:
- net +3V3: now also J3.8 (Pin_8), C15.2, C16.2, C8.2, J4.8 (Pin_8), J7.8 (Pin_8), J8.8 (Pin_8), R10.2, R15.2, R16.2, R17.2, R18.2, R19.2, R20.2, R5.2, R6.2, R7.2, R8.2, R9.2, U2.5 (AVDD), U2.8 (DVDD), U3.5 (AVDD), U3.8 (DVDD), U4.5 (AVDD), U4.8 (DVDD)
- net BIAS: now also J2.1 (Pin_1), J5.1 (Pin_1), J6.1 (Pin_1), R11.2, R13.2, R3.2, U2.2 (BIAS), U3.2 (BIAS), U4.2 (BIAS)
- net GNDREF: now also J3.7 (Pin_7), C11.2, C12.1, C14.2, C15.1, C16.1, C4.1, C6.2, C8.1, C9.1, J4.7 (Pin_7), J7.7 (Pin_7), J8.7 (Pin_7), U2.1 (AGND), U2.14 (DGND), U3.1 (AGND), U3.14 (DGND), U4.1 (AGND), U4.14 (DGND)
- net SCK: now reaches U1.10 (SCK)
- net SCK: now also J3.4 (Pin_4), J4.4 (Pin_4), J7.4 (Pin_4), J8.4 (Pin_4), R17.1, R18.1, R7.1, R8.1, U2.10 (SCK), U3.10 (SCK), U4.10 (SCK)
- net SDO: now reaches U1.11 (SDO)
- net SDO: now also J3.5 (Pin_5), J4.5 (Pin_5), J7.5 (Pin_5), J8.5 (Pin_5), U2.11 (SDO), U3.11 (SDO), U4.11 (SDO)
- net SDI: now reaches U1.12 (SDI)
- net SDI: now also J3.6 (Pin_6), J4.6 (Pin_6), J7.6 (Pin_6), J8.6 (Pin_6), R15.1, R16.1, R5.1, R6.1, U2.12 (SDI), U3.12 (SDI), U4.12 (SDI)
- net ~FAULT: now reaches U1.13 (~FAULT)
- net ~FAULT: now also J3.2 (Pin_2), J4.2 (Pin_2), J7.2 (Pin_2), J8.2 (Pin_2), U2.13 (~FAULT), U3.13 (~FAULT), U4.13 (~FAULT)
- net ~DRDY: now reaches U1.7 (~DRDY)
- net ~DRDY: now also J3.1 (Pin_1), J4.1 (Pin_1), J7.1 (Pin_1), J8.1 (Pin_1), U2.7 (~DRDY), U3.7 (~DRDY), U4.7 (~DRDY)
- net ~CS: now reaches U1.9 (~CS)
- net ~CS: now also J3.3 (Pin_3), J4.3 (Pin_3), J7.3 (Pin_3), J8.3 (Pin_3), R10.1, R19.1, R20.1, R9.1, U2.9 (~CS), U3.9 (~CS), U4.9 (~CS)
- new net: C4.2, C5.1, R3.1, U2.3 (T-)
- new net: C5.2, C6.1, R4.1, U2.4 (T+)
- new net: J2.2 (Pin_2), R4.2
- new net: C10.1, C9.2, R11.1, U3.3 (T-)
- new net: C10.2, C11.1, R12.1, U3.4 (T+)
- new net: J5.2 (Pin_2), R12.2
- new net: C12.2, C13.1, R13.1, U4.3 (T-)
- new net: C13.2, C14.1, R14.1, U4.4 (T+)
- new net: J6.2 (Pin_2), R14.2
Other:
- moved on the sheet: C1, C2, C3, C7, J1, R1, R2, U1
