File: PCB files/PayloadBoard/Payload2020/Payload2020A.sch (KiCad schematic (older format))
At the start: 3 parts, among them U1 Teensy3.6, U2 ArduCam, U3 HX711_Breakout

Commit message: -Added 20 pin connector to connect Board A to board B
Parts:
- removed U3: HX711_Breakout, Payload:HX711_Breakout, symbol PayloadBoard:HX711_Breakout
- added J?: BridgeConn, symbol Connector_Generic:Conn_02x10_Counter_Clockwise
- added U?: HX711_Breakout, symbol PayloadBoard:HX711_Breakout
Connections:
- wire segments 16 -> 23
Other:
- note added: "Load Cell ADC"
- moved on the sheet: U1, U2

Commit message: -Added connector to Board B -Added descriptive i2c local net names
Connections:
- net labels added: Ardu_SCL, Ardu_SDA, Berry_SCL, Berry_SDA
- net labels removed: SCL0, SDA0
- wire segments 23 -> 21
Other:
- moved on the sheet: U2, U?
Changed lines of the file:
@@
 EESchema Schematic File Version 4
-LIBS:Payload2020A-cache
-EELAYER 29 0
+EELAYER 30 0
 EELAYER END
 $Descr A4 11693 8268
@@
 L PayloadBoard:ArduCam U2
 U 1 1 5E4A2FC8
-P 9990 5810
-F 0 "U2" H 9990 6225 50  0000 C CNN
-F 1 "ArduCam" H 9990 6134 50  0000 C CNN
-F 2 "Payload:ArduCam" H 9840 5860 50  0001 C CNN
-F 3 "" H 9840 5860 50  0001 C CNN
-	1    9990 5810
-	-1   0    0    -1
+P 3380 4510
+F 0 "U2" H 3380 4925 50  0000 C CNN
+F 1 "ArduCam" H 3380 4834 50  0000 C CNN
+F 2 "Payload:ArduCam" H 3230 4560 50  0001 C CNN
+F 3 "" H 3230 4560 50  0001 C CNN
+	1    3380 4510
+	1    0    0    -1
 $EndComp
 $Comp
@@
 L power:GNDREF #PWR010
 U 1 1 5E5231F1
-P 9600 5660
-F 0 "#PWR010" H 9600 5410 50  0001 C CNN
-F 1 "GNDREF" H 9605 5487 50  0001 C CNN
-F 2 "" H 9600 5660 50  0001 C CNN
-F 3 "" H 9600 5660 50  0001 C CNN
-	1    9600 5660
-	0    1    -1   0
+P 3770 4360
+F 0 "#PWR010" H 3770 4110 50  0001 C CNN
+F 1 "GNDREF" H 3775 4187 50  0001 C CNN
+F 2 "" H 3770 4360 50  0001 C CNN
+F 3 "" H 3770 4360 50  0001 C CNN
+	1    3770 4360
+	0    -1   -1   0
 $EndComp
 Wire Wire Line
-	9640 5660 9600 5660
+	3730 4360 3770 4360
 $Comp
 L power:GNDREF #PWR03
@@
 L power:+3V3 #PWR01
 U 1 1 5E525372
-P 4640 2670
-F 0 "#PWR01" H 4640 2520 50  0001 C CNN
-F 1 "+3V3" H 4655 2843 50  0000 C CNN
-F 2 "" H 4640 2670 50  0001 C CNN
-F 3 "" H 4640 2670 50  0001 C CNN
-	1    4640 2670
+P 4840 2670
+F 0 "#PWR01" H 4840 2520 50  0001 C CNN
+F 1 "+3V3" H 4855 2843 50  0000 C CNN
+F 2 "" H 4840 2670 50  0001 C CNN
+F 3 "" H 4840 2670 50  0001 C CNN
+	1    4840 2670
 	1    0    0    -1
 $EndComp
 Wire Wire Line
-	4640 2670 5090 2670
+	4840 2670 5090 2670
 $Comp
 L power:GNDREF #PWR04
@@
 L power:+3V3 #PWR09
 U 1 1 5E52F8CC
-P 9370 5760
-F 0 "#PWR09" H 9370 5610 50  0001 C CNN
-F 1 "+3V3" H 9385 5933 50  0000 C CNN
-F 2 "" H 9370 5760 50  0001 C CNN
-F 3 "" H 9370 5760 50  0001 C CNN
-	1    9370 5760
-	1    0    0    -1
+P 4000 4460
+F 0 "#PWR09" H 4000 4310 50  0001 C CNN
+F 1 "+3V3" H 4015 4633 50  0000 C CNN
+F 2 "" H 4000 4460 50  0001 C CNN
+F 3 "" H 4000 4460 50  0001 C CNN
+	1    4000 4460
+	-1   0    0    -1
 $EndComp
 Wire Wire Line
-	9370 5760 9640 5760
-Text Label 7590 5470 2    50   ~ 0
-SCL0
-Text Label 7590 5570 2    50   ~ 0
-SDA0
-Text Label 9440 5860 0    50   ~ 0
-SDA0
-Text Label 9440 5960 0    50   ~ 0
-SCL0
-Wire Wire Line
-	9440 5960 9640 5960
-Wire Wire Line
-	9440 5860 9640 5860
-Wire Wire Line
-	7590 5570 7390 5570
-Wire Wire Line
-	7390 5470 7590 5470
-Text Notes 2460 5450 0    50   ~ 0
+	4000 4460 3730 4460
+Text Label 4080 4560 2    50   ~ 0
+Ardu_SDA
+Text Label 4080 4660 2    50   ~ 0
+Ardu_SCL
+Text Notes 3650 5000 2    50   ~ 0
 Load Cell ADC
 $Comp
 L PayloadBoard:HX711_Breakout U?
 U 1 1 5E539E03
-P 2750 6120
-F 0 "U?" H 2750 6495 50  0000 C CNN
-F 1 "HX711_Breakout" H 2750 6404 50  0000 C CNN
-F 2 "" H 2750 6520 50  0001 C CNN
-F 3 "" H 2750 6520 50  0001 C CNN
-	1    2750 6120
-	1    0    0    -1
+P 3400 5460
+F 0 "U?" H 3400 5835 50  0000 C CNN
+F 1 "HX711_Breakout" H 3400 5744 50  0000 C CNN
+F 2 "" H 3400 5860 50  0001 C CNN
+F 3 "" H 3400 5860 50  0001 C CNN
+	1    3400 5460
+	-1   0    0    -1
 $EndComp
 $Comp
 L power:GNDREF #PWR?
 U 1 1 5E534372
-P 3130 6070
-F 0 "#PWR?" H 3130 5820 50  0001 C CNN
-F 1 "GNDREF" H 3135 5897 50  0001 C CNN
-F 2 "" H 3130 6070 50  0001 C CNN
-F 3 "" H 3130 6070 50  0001 C CNN
-	1    3130 6070
-	0    -1   -1   0
+P 3020 5410
+F 0 "#PWR?" H 3020 5160 50  0001 C CNN
+F 1 "GNDREF" H 3025 5237 50  0001 C CNN
+F 2 "" H 3020 5410 50  0001 C CNN
+F 3 "" H 3020 5410 50  0001 C CNN
+	1    3020 5410
+	0    1    -1   0
 $EndComp
 Wire Wire Line
-	3100 6070 3130 6070
+	3050 5410 3020 5410
 $Comp
 L power:+3V3 #PWR?
 U 1 1 5E5358F8
-P 3320 6370
-F 0 "#PWR?" H 3320 6220 50  0001 C CNN
-F 1 "+3V3" H 3335 6543 50  0000 C CNN
-F 2 "" H 3320 6370 50  0001 C CNN
-F 3 "" H 3320 6370 50  0001 C CNN
-	1    3320 6370
-	1    0    0    -1
+P 2830 5710
+F 0 "#PWR?" H 2830 5560 50  0001 C CNN
+F 1 "+3V3" H 2845 5883 50  0000 C CNN
+F 2 "" H 2830 5710 50  0001 C CNN
+F 3 "" H 2830 5710 50  0001 C CNN
+	1    2830 5710
+	-1   0    0    -1
 $EndComp
 Wire Wire Line
-	3320 6370 3100 6370
+	2830 5710 3050 5710
 $Comp
 L Connector_Generic:Conn_02x10_Counter_Clockwise J?
 U 1 1 5E53BD04
-P 1670 5970
-F 0 "J?" H 1720 6587 50  0000 C CNN
-F 1 "BridgeConn" H 1720 6496 50  0000 C CNN
-F 2 "" H 1670 5970 50  0001 C CNN
-F 3 "~" H 1670 5970 50  0001 C CNN
-	1    1670 5970
+P 8690 2500
+F 0 "J?" H 8740 3117 50  0000 C CNN
+F 1 "BridgeConn" H 8740 3026 50  0000 C CNN
+F 2 "" H 8690 2500 50  0001 C CNN
+F 3 "~" H 8690 2500 50  0001 C CNN
+	1    8690 2500
 	1    0    0    -1
 $EndComp
+Text Label 8090 2100 0    50   ~ 0
+Berry_SDA
+Wire Wire Line
+	8090 2100 8490 2100
+Text Label 8090 2200 0    50   ~ 0
+Berry_SCL
+Wire Wire Line
+	8090 2200 8490 2200
 Wire Wire Line
-	1970 6470 2400 6470
+	4080 4560 3730 4560
 Wire Wire Line
-	2400 6370 1970 6370
+	4080 4660 3730 4660
+Text Label 7740 5470 2    50   ~ 0
+Ardu_SDA
+Text Label 7740 5570 2    50   ~ 0
+Ardu_SCL
 Wire Wire Line
-	1970 6270 2400 6270
+	7390 5470 7740 5470
 Wire Wire Line
-	2400 6170 1970 6170
+	7390 5570 7740 5570
+Text Label 4720 4670 0    50   ~ 0
+Ardu_SDA
+Text Label 4720 4570 0    50   ~ 0
+Ardu_SCL
 Wire Wire Line
-	1970 6070 2400 6070
+	4720 4670 5090 4670
 Wire Wire Line
-	2400 5970 1970 5970
+	4720 4570 5090 4570
 $EndSCHEMATC

Commit message: Changes to PayloadBoard A schematic -Added 3v3 and 5v regulation -Created corresponding symbols for regulators -Added net names for i2c and SPI connections
Parts:
- added J?: BATTERY, symbol Connector:Conn_01x02_Female
- added U?: AP7370-50W5-7, symbol PayloadBoard:AP7370-50W5-7
- added U?: AP2210N-5.0TRG1, symbol PayloadBoard:AP2210N-5.0TRG1
Connections:
- net labels added: +3.3VA, +5V, Ardu_CS, Ardu_MISO, Ardu_MOSI, Ardu_SCK, HX_OUT
- wire segments 21 -> 42
- no-connect marks 0 -> 2
Other:
- note added: "+"
- note added: "-"
- note added: "2sXp LiON"
- note added: "3V3A - Power to Xbee from battery\n3V3 - Power to ArduCam, HX711, and BerryIMU from Teensy"
- note added: "6-8.4V IN"
- moved on the sheet: U2, U?

Commit message: Payload Board B changes -Added xbee and berry GPS signal pin local nets -Added power and gnd flags to berry and xbee
Connections:
- wire segments 42 -> 43
Changed lines of the file:
@@
 Text Notes 7520 760  0    79   ~ 0
 3V3A - Power to Xbee from battery\n3V3 - Power to ArduCam, HX711, and BerryIMU from Teensy
+$Comp
+L power:+3.3VA #PWR?
+U 1 1 5E5BD94E
+P 7900 2300
+F 0 "#PWR?" H 7900 2150 50  0001 C CNN
+F 1 "+3.3VA" H 7915 2473 50  0000 C CNN
+F 2 "" H 7900 2300 50  0001 C CNN
+F 3 "" H 7900 2300 50  0001 C CNN
+	1    7900 2300
+	1    0    0    -1
+$EndComp
+Wire Wire Line
+	8490 2300 7900 2300
 $EndSCHEMATC

Commit message: Removed 5V regulator Stepped input voltage down to that of a 1s battery pack Added internal parallite battery connection
Parts:
- removed U?: AP2210N-5.0TRG1, symbol PayloadBoard:AP2210N-5.0TRG1
- added J?: BATTERY, symbol Connector:Conn_01x02_Female
Connections:
- wire segments 43 -> 38
Other:
- note added: "1sXp LiON"
- note added: "3-4.2V"
- note added: "<--- from boost converter"
- note added: "Add Boost converter here"
- note added: "Add switching circuit here"
- note added: "Flat LiPo 180 mAh"
- note removed: "2sXp LiON"
- note removed: "6-8.4V IN"
Changed lines of the file:
@@
 L Connector:Conn_01x02_Female J?
 U 1 1 5E5498CC
-P 1220 1360
-F 0 "J?" H 1112 1545 50  0000 C CNN
-F 1 "BATTERY" H 1112 1454 50  0000 C CNN
-F 2 "" H 1220 1360 50  0001 C CNN
-F 3 "~" H 1220 1360 50  0001 C CNN
-	1    1220 1360
-	-1   0    0    -1
-$EndComp
-Text Notes 1120 1390 0    50   ~ 0
+P 1120 1130
+F 0 "J?" H 1012 1315 50  0000 C CNN
+F 1 "BATTERY" H 1012 1224 50  0000 C CNN
+F 2 "" H 1120 1130 50  0001 C CNN
+F 3 "~" H 1120 1130 50  0001 C CNN
+	1    1120 1130
+	-1   0    0    -1
+$EndComp
+Text Notes 1010 1170 0    50   ~ 0
 +
-Text Notes 1120 1490 0    50   ~ 0
+Text Notes 1010 1270 0    50   ~ 0
 -
-$Comp
-L power:GNDREF #PWR?
-U 1 1 5E54B0A0
-P 1530 1460
-F 0 "#PWR?" H 1530 1210 50  0001 C CNN
-F 1 "GNDREF" H 1535 1287 50  0001 C CNN
-F 2 "" H 1530 1460 50  0001 C CNN
-F 3 "" H 1530 1460 50  0001 C CNN
-	1    1530 1460
-	1    0    0    -1
-$EndComp
-Wire Wire Line
-	1420 1460 1530 1460
-$Comp
-L PayloadBoard:AP7370-50W5-7 U?
-U 1 1 5E54C67E
-P 2660 1560
-F 0 "U?" H 2660 1985 50  0000 C CNN
-F 1 "AP7370-50W5-7" H 2660 1894 50  0000 C CNN
-F 2 "" H 2610 1910 50  0001 C CNN
-F 3 "https://www.diodes.com/assets/Datasheets/AP7370.pdf" H 2610 1910 50  0001 C CNN
-	1    2660 1560
-	1    0    0    -1
-$EndComp
-NoConn ~ 3010 1660
-NoConn ~ 2310 1760
-$Comp
-L power:GNDREF #PWR?
-U 1 1 5E54D5EC
-P 2260 1560
-F 0 "#PWR?" H 2260 1310 50  0001 C CNN
-F 1 "GNDREF" H 2265 1387 50  0001 C CNN
-F 2 "" H 2260 1560 50  0001 C CNN
-F 3 "" H 2260 1560 50  0001 C CNN
-	1    2260 1560
-	1    0    0    -1
-$EndComp
-Wire Wire Line
-	2260 1560 2310 1560
-Text Notes 1510 1360 0    50   ~ 0
-6-8.4V IN
-Text Notes 1020 1640 0    50   ~ 0
-2sXp LiON
+Text Notes 1410 1130 0    50   ~ 0
+3-4.2V
+Text Notes 890  1350 0    50   ~ 0
+1sXp LiON
 Wire Wire Line
 	2920 4130 4490 4130
@@
 Wire Wire Line
 	4590 1370 5090 1370
-Wire Wire Line
-	1420 1360 1940 1360
-$Comp
-L PayloadBoard:AP2210N-5.0TRG1 U?
-U 1 1 5E598D25
-P 2640 2440
-F 0 "U?" H 2640 2755 50  0000 C CNN
-F 1 "AP2210N-5.0TRG1" H 2640 2664 50  0000 C CNN
-F 2 "" H 2490 2640 50  0001 C CNN
-F 3 "" H 2490 2640 50  0001 C CNN
-	1    2640 2440
-	1    0    0    -1
-$EndComp
-Wire Wire Line
-	1940 1360 1940 2390
-Connection ~ 1940 1360
-Wire Wire Line
-	1940 1360 2310 1360
-$Comp
-L power:GNDREF #PWR?
-U 1 1 5E59A364
-P 2640 2790
-F 0 "#PWR?" H 2640 2540 50  0001 C CNN
-F 1 "GNDREF" H 2645 2617 50  0001 C CNN
-F 2 "" H 2640 2790 50  0001 C CNN
-F 3 "" H 2640 2790 50  0001 C CNN
-	1    2640 2790
-	1    0    0    -1
-$EndComp
-Wire Wire Line
-	2640 2790 2640 2740
-$Comp
-L power:+5V #PWR?
-U 1 1 5E59BE17
-P 3140 2390
-F 0 "#PWR?" H 3140 2240 50  0001 C CNN
-F 1 "+5V" H 3155 2563 50  0000 C CNN
-F 2 "" H 3140 2390 50  0001 C CNN
-F 3 "" H 3140 2390 50  0001 C CNN
-	1    3140 2390
-	1    0    0    -1
-$EndComp
-Wire Wire Line
-	3040 2390 3140 2390
-Wire Wire Line
-	1940 2390 2240 2390
 $Comp
 L power:+5V #PWR?
@@
 L power:+3.3VA #PWR?
 U 1 1 5E5B7BCF
-P 3190 1460
-F 0 "#PWR?" H 3190 1310 50  0001 C CNN
-F 1 "+3.3VA" H 3205 1633 50  0000 C CNN
-F 2 "" H 3190 1460 50  0001 C CNN
-F 3 "" H 3190 1460 50  0001 C CNN
-	1    3190 1460
-	1    0    0    -1
-$EndComp
-Wire Wire Line
-	3010 1460 3190 1460
+P 3680 2650
+F 0 "#PWR?" H 3680 2500 50  0001 C CNN
+F 1 "+3.3VA" H 3695 2823 50  0000 C CNN
+F 2 "" H 3680 2650 50  0001 C CNN
+F 3 "" H 3680 2650 50  0001 C CNN
+	1    3680 2650
+	1    0    0    -1
+$EndComp
 Text Label 4680 1770 0    50   ~ 0
 Berry_SDA
@@
 Wire Wire Line
 	8490 2300 7900 2300
+Text Notes 3120 1580 0    50   ~ 0
+Add Boost converter here
+Wire Wire Line
+	3500 2650 3680 2650
+Wire Wire Line
+	2750 2750 2800 2750
+$Comp
+L power:GNDREF #PWR?
+U 1 1 5E54D5EC
+P 2750 2750
+F 0 "#PWR?" H 2750 2500 50  0001 C CNN
+F 1 "GNDREF" H 2755 2577 50  0001 C CNN
+F 2 "" H 2750 2750 50  0001 C CNN
+F 3 "" H 2750 2750 50  0001 C CNN
+	1    2750 2750
+	1    0    0    -1
+$EndComp
+NoConn ~ 2800 2950
+NoConn ~ 3500 2850
+$Comp
+L PayloadBoard:AP7370-50W5-7 U?
+U 1 1 5E54C67E
+P 3150 2750
+F 0 "U?" H 3150 3175 50  0000 C CNN
+F 1 "AP7370-50W5-7" H 3150 3084 50  0000 C CNN
+F 2 "" H 3100 3100 50  0001 C CNN
+F 3 "https://www.diodes.com/assets/Datasheets/AP7370.pdf" H 3100 3100 50  0001 C CNN
+	1    3150 2750
+	1    0    0    -1
+$EndComp
+$Comp
+L Connector:Conn_01x02_Female J?
+U 1 1 5E59244E
+P 1100 1880
+F 0 "J?" H 992 2065 50  0000 C CNN
+F 1 "BATTERY" H 992 1974 50  0000 C CNN
+F 2 "" H 1100 1880 50  0001 C CNN
+F 3 "~" H 1100 1880 50  0001 C CNN
+	1    1100 1880
+	-1   0    0    -1
+$EndComp
+Text Notes 990  1910 0    50   ~ 0
++
+Text Notes 990  2010 0    50   ~ 0
+-
+Text Notes 630  2120 0    50   ~ 0
+Flat LiPo 180 mAh
+Wire Wire Line
+	1320 1230 1430 1230
+$Comp
+L power:GNDREF #PWR?
+U 1 1 5E54B0A0
+P 1430 1230
+F 0 "#PWR?" H 1430 980 50  0001 C CNN
+F 1 "GNDREF" H 1435 1057 50  0001 C CNN
+F 2 "" H 1430 1230 50  0001 C CNN
+F 3 "" H 1430 1230 50  0001 C CNN
+	1    1430 1230
+	1    0    0    -1
+$EndComp
+$Comp
+L power:GNDREF #PWR?
+U 1 1 5E594677
+P 1410 1980
+F 0 "#PWR?" H 1410 1730 50  0001 C CNN
+F 1 "GNDREF" H 1415 1807 50  0001 C CNN
+F 2 "" H 1410 1980 50  0001 C CNN
+F 3 "" H 1410 1980 50  0001 C CNN
+	1    1410 1980
+	1    0    0    -1
+$EndComp
+Wire Wire Line
+	1410 1980 1300 1980
+Text Notes 1820 1570 0    50   ~ 0
+Add switching circuit here
+Text Notes 7620 4640 0    50   ~ 0
+<--- from boost converter
+Text Notes 1400 1850 0    50   ~ 0
+3-4.2V
 $EndSCHEMATC

Commit message: Created boost converter symbol Added 5V boost converter circuit Selected footprints for caps and IC's
Parts:
- removed J?: BATTERY, symbol Connector:Conn_01x02_Female
- added C1, C2: 1uF, Capacitor_SMD:C_1206_3216Metric, symbol Device:C_Small
- added C3: 22uF, Capacitor_SMD:C_1206_3216Metric, symbol Device:C_Small
- added L1: 4.7uH, symbol Device:L
- added U5: TPS613222ADBVR, Package_TO_SOT_SMD:SOT-23-5, symbol PayloadBoard:TPS613222ADBVR
- U3: renamed from U?; footprint (none) -> Payload:HX711_Breakout
- U4: renamed from U?; footprint (none) -> Package_TO_SOT_SMD:SOT-23-5
- gave numbers to parts that had none: 2
Connections:
- wire segments 38 -> 53
- no-connect marks 2 -> 4
Other:
- note added: "3.3V dedicated to Xbee"
- note removed: "Add Boost converter here"
- note removed: "Add switching circuit here"
- note removed: "Flat LiPo 180 mAh"

Commit message: -began footprint for berryIMU -Added XBEE sparkfun footprints from github -Added xbee and gps net connection to connector on board A
Parts:
- J2: symbol Connector_Generic:Conn_02x10_Counter_Clockwise -> Connector_Generic:Conn_01x09
- L1: footprint (none) -> Inductor_SMD:L_Taiyo-Yuden_MD-5050
Connections:
- net labels added: RX_GPS, TX_GPS, XBEE_CTS, XBEE_DIN, XBEE_DOUT, XBEE_RTS
- wire segments 53 -> 66
Other:
- moved on the sheet: U1, U2, U3

Commit message: Updated boost converter L and C values according to datasheet
Parts:
- added C4: 10uF, Capacitor_SMD:C_1206_3216Metric, symbol Device:C_Small
- C3: value 22uF -> 10uF
- L1: value 4.7uH -> 2.2uH; footprint Inductor_SMD:L_Taiyo-Yuden_MD-5050 -> Inductor_SMD:L_1210_3225Metric
Connections:
- net labels added: HX_CLK
- wire segments 66 -> 70
Other:
- note added: "3.3VA dedicated to Xbee"
- note removed: "3.3V dedicated to Xbee"
Changed lines of the file:
@@
 Wire Wire Line
 	4660 5920 5080 5920
-Text Label 9060 3450 0    50   ~ 0
+Text Label 8950 3450 0    50   ~ 0
 HX_OUT
-Wire Wire Line
-	9060 3450 9360 3450
 Text Label 4670 2120 0    50   ~ 0
 HX_OUT
@@
 Wire Wire Line
 	2300 1030 2350 1030
-$Comp
-L power:+3.3VA #PWR016
-U 1 1 5E5B7BCF
-P 3360 930
-F 0 "#PWR016" H 3360 780 50  0001 C CNN
-F 1 "+3.3VA" H 3375 1103 50  0000 C CNN
-F 2 "" H 3360 930 50  0001 C CNN
-F 3 "" H 3360 930 50  0001 C CNN
-	1    3360 930
-	1    0    0    -1
-$EndComp
 Wire Wire Line
 	2350 830  2050 830
@@
 P 2060 1790
 F 0 "L1" V 1879 1790 50  0000 C CNN
-F 1 "4.7uH" V 1970 1790 50  0000 C CNN
-F 2 "Inductor_SMD:L_Taiyo-Yuden_MD-5050" H 2060 1790 50  0001 C CNN
+F 1 "2.2uH" V 1970 1790 50  0000 C CNN
+F 2 "Inductor_SMD:L_1210_3225Metric" H 2060 1790 50  0001 C CNN
 F 3 "~" H 2060 1790 50  0001 C CNN
 	1    2060 1790
@@
 	1    0    0    -1
 $EndComp
-Wire Wire Line
-	3290 2070 3290 2020
 $Comp
 L power:+5V #PWR017
 U 1 1 5E5E1BBE
-P 3480 1790
-F 0 "#PWR017" H 3480 1640 50  0001 C CNN
-F 1 "+5V" H 3495 1963 50  0000 C CNN
-F 2 "" H 3480 1790 50  0001 C CNN
-F 3 "" H 3480 1790 50  0001 C CNN
-	1    3480 1790
+P 3880 1790
+F 0 "#PWR017" H 3880 1640 50  0001 C CNN
+F 1 "+5V" H 3895 1963 50  0000 C CNN
+F 2 "" H 3880 1790 50  0001 C CNN
+F 3 "" H 3880 1790 50  0001 C CNN
+	1    3880 1790
 	1    0    0    -1
 $EndComp
@@
 Wire Wire Line
 	1530 830  1070 830
-Text Notes 3250 710  0    50   ~ 0
-3.3V dedicated to Xbee
+Text Notes 3360 560  0    50   ~ 0
+3.3VA dedicated to Xbee
 $Comp
 L Device:C_Small C3
 U 1 1 5E5E74CE
-P 3290 1920
-F 0 "C3" H 3382 1966 50  0000 L CNN
-F 1 "22uF" H 3382 1875 50  0000 L CNN
-F 2 "Capacitor_SMD:C_1206_3216Metric" H 3290 1920 50  0001 C CNN
-F 3 "~" H 3290 1920 50  0001 C CNN
-	1    3290 1920
-	1    0    0    -1
-$EndComp
-Wire Wire Line
-	3100 1790 3290 1790
+P 3290 1890
+F 0 "C3" H 3382 1936 50  0000 L CNN
+F 1 "10uF" H 3382 1845 50  0000 L CNN
+F 2 "Capacitor_SMD:C_1206_3216Metric" H 3290 1890 50  0001 C CNN
+F 3 "~" H 3290 1890 50  0001 C CNN
+	1    3290 1890
+	1    0    0    -1
+$EndComp
 $Comp
 L Device:C_Small C2
 U 1 1 5E5E7EDC
-P 3270 1120
-F 0 "C2" H 3362 1166 50  0000 L CNN
-F 1 "1uF" H 3362 1075 50  0000 L CNN
-F 2 "Capacitor_SMD:C_1206_3216Metric" H 3270 1120 50  0001 C CNN
-F 3 "~" H 3270 1120 50  0001 C CNN
-	1    3270 1120
+P 3270 1020
+F 0 "C2" H 3362 1066 50  0000 L CNN
+F 1 "1uF" H 3362 975 50  0000 L CNN
+F 2 "Capacitor_SMD:C_1206_3216Metric" H 3270 1020 50  0001 C CNN
+F 3 "~" H 3270 1020 50  0001 C CNN
+	1    3270 1020
 	1    0    0    -1
 $EndComp
@@
 Wire Wire Line
 	2050 1120 2050 1070
-Wire Wire Line
-	3050 930  3270 930
-Wire Wire Line
-	3270 1020 3270 930
-Connection ~ 3270 930
-Wire Wire Line
-	3270 930  3360 930
 $Comp
 L power:GNDREF #PWR014
 U 1 1 5E5F64DE
-P 3270 1280
-F 0 "#PWR014" H 3270 1030 50  0001 C CNN
-F 1 "GNDREF" H 3275 1107 50  0001 C CNN
-F 2 "" H 3270 1280 50  0001 C CNN
-F 3 "" H 3270 1280 50  0001 C CNN
-	1    3270 1280
-	1    0    0    -1
-$EndComp
-Wire Wire Line
-	3270 1280 3270 1220
-Wire Wire Line
-	3290 1820 3290 1790
-Connection ~ 3290 1790
-Wire Wire Line
-	3290 1790 3480 1790
+P 3270 1180
+F 0 "#PWR014" H 3270 930 50  0001 C CNN
+F 1 "GNDREF" H 3275 1007 50  0001 C CNN
+F 2 "" H 3270 1180 50  0001 C CNN
+F 3 "" H 3270 1180 50  0001 C CNN
+	1    3270 1180
+	1    0    0    -1
+$EndComp
+Wire Wire Line
+	3270 1180 3270 1120
 Text Label 9080 2450 0    50   ~ 0
 XBEE_DOUT
@@
 Wire Wire Line
 	4220 4880 4480 4880
+$Comp
+L Device:C_Small C4
+U 1 1 5E606AD0
+P 3650 1890
+F 0 "C4" H 3742 1936 50  0000 L CNN
+F 1 "10uF" H 3742 1845 50  0000 L CNN
+F 2 "Capacitor_SMD:C_1206_3216Metric" H 3650 1890 50  0001 C CNN
+F 3 "~" H 3650 1890 50  0001 C CNN
+	1    3650 1890
+	1    0    0    -1
+$EndComp
+Connection ~ 3650 1790
+$Comp
+L power:GNDREF #PWR021
+U 1 1 5E60B177
+P 3650 2070
+F 0 "#PWR021" H 3650 1820 50  0001 C CNN
+F 1 "GNDREF" H 3655 1897 50  0001 C CNN
+F 2 "" H 3650 2070 50  0001 C CNN
+F 3 "" H 3650 2070 50  0001 C CNN
+	1    3650 2070
+	1    0    0    -1
+$EndComp
+Wire Wire Line
+	3650 1990 3650 2070
+Wire Wire Line
+	3100 1790 3290 1790
+Connection ~ 3290 1790
+Wire Wire Line
+	3290 1790 3650 1790
+Wire Wire Line
+	3290 1990 3290 2070
+Wire Wire Line
+	3650 1790 3880 1790
+Wire Wire Line
+	3270 920  3270 830
+$Comp
+L power:+3.3VA #PWR016
+U 1 1 5E5B7BCF
+P 3360 830
+F 0 "#PWR016" H 3360 680 50  0001 C CNN
+F 1 "+3.3VA" H 3375 1003 50  0000 C CNN
+F 2 "" H 3360 830 50  0001 C CNN
+F 3 "" H 3360 830 50  0001 C CNN
+	1    3360 830
+	1    0    0    -1
+$EndComp
+Wire Wire Line
+	3270 830  3360 830
+Wire Wire Line
+	3050 930  3050 830
+Wire Wire Line
+	3050 830  3270 830
+Connection ~ 3270 830
+Text Label 4670 2220 0    50   ~ 0
+HX_CLK
+Wire Wire Line
+	4670 2220 5080 2220
+Text Label 8950 3350 0    50   ~ 0
+HX_CLK
+Wire Wire Line
+	8950 3350 9360 3350
+Wire Wire Line
+	8950 3450 9360 3450
 $EndSCHEMATC
