File: PCB files/PayloadBoard/Payload2020/Payload2020A.sch (KiCad schematic (older format))
At the start: 12 parts, among them J1 BATTERY, J2 BridgeConn, U1 Teensy3.6, U2 ArduCam, U3 HX711_Breakout, U4 AP7370-50W5-7, U5 TPS613222ADBVR

Commit message: Arranged more components on board -Drew board edges for board B -Added User controlled LEDs
Parts:
- added D1, D2: LED, symbol Device:LED
- added J3: LoadCell, symbol Connector:Conn_01x04_Female
- added Q1, Q2: Q_NMOS_GSD, symbol Device:Q_NMOS_GSD
- added R1, R2, R4, R5: 10k, symbol Device:R_US
- added R3, R6: 100, symbol Device:R_US
- J1: footprint (none) -> Connector_JST:JST_EH_S2B-EH_1x02_P2.50mm_Horizontal
Connections:
- net labels added: USR_LED1, USR_LED2
- wire segments 70 -> 102
- no-connect marks 4 -> 6
Other:
- note added: "*"
- note added: "USER CONTROLLED LEDS"
- note added: "Voltage Boost/Regulation"
- note removed: "3.3VA dedicated to Xbee"
- moved on the sheet: U3

Commit message: Changed board sizes based on payload bay dimensions Changed battery connector to JST XH
Parts:
- J1: footprint Connector_JST:JST_EH_S2B-EH_1x02_P2.50mm_Horizontal -> Connector_JST:JST_XH_B2B-XH-AM_1x02_P2.50mm_Vertical
Changed lines of the file:
@@
 F 0 "J1" H 732 1295 50  0000 C CNN
 F 1 "BATTERY" H 732 1204 50  0000 C CNN
-F 2 "Connector_JST:JST_EH_S2B-EH_1x02_P2.50mm_Horizontal" H 840 1110 50  0001 C CNN
+F 2 "Connector_JST:JST_XH_B2B-XH-AM_1x02_P2.50mm_Vertical" H 840 1110 50  0001 C CNN
 F 3 "~" H 840 1110 50  0001 C CNN
 	1    840  1110

Commit message: -Selected all footprints -Began routing Board A
Parts:
- added SW1: SW_SPST, Payload:GW12RCH, symbol Switch:SW_SPST
- D1, D2: footprint (none) -> LED_SMD:LED_1206_3216Metric
- J2: footprint (none) -> Connector_JST:JST_SH_BM09B-SRSS-TB_1x09-1MP_P1.00mm_Vertical
- J3: footprint (none) -> Connector_JST:JST_SH_BM04B-SRSS-TB_1x04-1MP_P1.00mm_Vertical
- Q1, Q2: footprint (none) -> Package_TO_SOT_SMD:SOT-23
- R1: value 10k -> 1k; footprint (none) -> Resistor_SMD:R_0805_2012Metric_Pad1.15x1.40mm_HandSolder
- R2: value 10k -> 100k; footprint (none) -> Resistor_SMD:R_0805_2012Metric_Pad1.15x1.40mm_HandSolder
- R3, R4, R5, R6: footprint (none) -> Resistor_SMD:R_0805_2012Metric_Pad1.15x1.40mm_HandSolder
Connections:
- wire segments 102 -> 103
Changed lines of the file:
@@
 F 0 "J2" H 9780 2767 50  0000 C CNN
 F 1 "BridgeConn" H 9780 2676 50  0000 C CNN
-F 2 "" H 9730 2150 50  0001 C CNN
+F 2 "Connector_JST:JST_SH_BM09B-SRSS-TB_1x09-1MP_P1.00mm_Vertical" H 9730 2150 50  0001 C CNN
 F 3 "~" H 9730 2150 50  0001 C CNN
 	1    9730 2150
@@
 U 1 1 5E5498CC
 P 840 1110
-F 0 "J1" H 732 1295 50  0000 C CNN
-F 1 "BATTERY" H 732 1204 50  0000 C CNN
+F 0 "J1" H 840 1280 50  0000 C CNN
+F 1 "BATTERY" H 840 1210 50  0000 C CNN
 F 2 "Connector_JST:JST_XH_B2B-XH-AM_1x02_P2.50mm_Vertical" H 840 1110 50  0001 C CNN
 F 3 "~" H 840 1110 50  0001 C CNN
@@
 Text Notes 730  1250 0    50   ~ 0
 -
-Text Notes 1130 1110 0    50   ~ 0
+Text Notes 1290 1110 2    50   ~ 0
 3-4.2V
 Text Notes 610  1330 0    50   ~ 0
@@
 $EndComp
 Wire Wire Line
-	1880 2070 1500 2070
-Wire Wire Line
-	1500 2070 1500 1110
-Connection ~ 1500 1110
-Wire Wire Line
-	1500 1110 1040 1110
+	1880 2070 1730 2070
+Wire Wire Line
+	1730 2070 1730 1110
 $Comp
 L Device:C_Small C3
@@
 Connection ~ 2020 1110
 Wire Wire Line
-	2020 1110 1500 1110
+	2020 1110 1730 1110
 $Comp
 L power:GNDREF #PWR011
@@
 F 0 "J3" H 10032 3695 50  0000 C CNN
 F 1 "LoadCell" H 10032 3786 50  0000 C CNN
-F 2 "" H 10140 4120 50  0001 C CNN
+F 2 "Connector_JST:JST_SH_BM04B-SRSS-TB_1x04-1MP_P1.00mm_Vertical" H 10140 4120 50  0001 C CNN
 F 3 "~" H 10140 4120 50  0001 C CNN
 	1    10140 4120
@@
 F 0 "D1" V 1619 6333 50  0000 R CNN
 F 1 "LED" V 1528 6333 50  0000 R CNN
-F 2 "" H 1580 6450 50  0001 C CNN
+F 2 "LED_SMD:LED_1206_3216Metric" H 1580 6450 50  0001 C CNN
 F 3 "~" H 1580 6450 50  0001 C CNN
 	1    1580 6450
@@
 F 0 "Q1" H 1686 6936 50  0000 L CNN
 F 1 "Q_NMOS_GSD" H 1686 6845 50  0000 L CNN
-F 2 "" H 1680 6990 50  0001 C CNN
+F 2 "Package_TO_SOT_SMD:SOT-23" H 1680 6990 50  0001 C CNN
 F 3 "~" H 1480 6890 50  0001 C CNN
 	1    1480 6890
@@
 P 1280 6450
 F 0 "R1" H 1348 6496 50  0000 L CNN
-F 1 "10k" H 1348 6405 50  0000 L CNN
-F 2 "" V 1320 6440 50  0001 C CNN
+F 1 "1k" H 1348 6405 50  0000 L CNN
+F 2 "Resistor_SMD:R_0805_2012Metric_Pad1.15x1.40mm_HandSolder" V 1320 6440 50  0001 C CNN
 F 3 "~" H 1280 6450 50  0001 C CNN
 	1    1280 6450
@@
 P 1280 7310
 F 0 "R2" H 1348 7356 50  0000 L CNN
-F 1 "10k" H 1348 7265 50  0000 L CNN
-F 2 "" V 1320 7300 50  0001 C CNN
+F 1 "100k" H 1348 7265 50  0000 L CNN
+F 2 "Resistor_SMD:R_0805_2012Metric_Pad1.15x1.40mm_HandSolder" V 1320 7300 50  0001 C CNN
 F 3 "~" H 1280 7310 50  0001 C CNN
 	1    1280 7310
@@
 Wire Wire Line
 	830  6890 1280 6890
-$Comp
-L Device:R_US R3
-U 1 1 5E623A5D
-P 1580 7310
-F 0 "R3" H 1648 7356 50  0000 L CNN
-F 1 "100" H 1648 7265 50  0000 L CNN
-F 2 "" V 1620 7300 50  0001 C CNN
-F 3 "~" H 1580 7310 50  0001 C CNN
-	1    1580 7310
-	1    0    0    -1
-$EndComp
 Wire Wire Line
 	1280 6890 1280 7160
@@
 F 0 "D2" V 3139 6363 50  0000 R CNN
 F 1 "LED" V 3048 6363 50  0000 R CNN
-F 2 "" H 3100 6480 50  0001 C CNN
+F 2 "LED_SMD:LED_1206_3216Metric" H 3100 6480 50  0001 C CNN
 F 3 "~" H 3100 6480 50  0001 C CNN
 	1    3100 6480
@@
 F 0 "Q2" H 3206 6966 50  0000 L CNN
 F 1 "Q_NMOS_GSD" H 3206 6875 50  0000 L CNN
-F 2 "" H 3200 7020 50  0001 C CNN
+F 2 "Package_TO_SOT_SMD:SOT-23" H 3200 7020 50  0001 C CNN
 F 3 "~" H 3000 6920 50  0001 C CNN
 	1    3000 6920
@@
 F 0 "R4" H 2868 6526 50  0000 L CNN
 F 1 "10k" H 2868 6435 50  0000 L CNN
-F 2 "" V 2840 6470 50  0001 C CNN
+F 2 "Resistor_SMD:R_0805_2012Metric_Pad1.15x1.40mm_HandSolder" V 2840 6470 50  0001 C CNN
 F 3 "~" H 2800 6480 50  0001 C CNN
 	1    2800 6480
@@
 F 0 "R5" H 2868 7386 50  0000 L CNN
 F 1 "10k" H 2868 7295 50  0000 L CNN
-F 2 "" V 2840 7330 50  0001 C CNN
+F 2 "Resistor_SMD:R_0805_2012Metric_Pad1.15x1.40mm_HandSolder" V 2840 7330 50  0001 C CNN
 F 3 "~" H 2800 7340 50  0001 C CNN
 	1    2800 7340
@@
 Wire Wire Line
 	2350 6920 2800 6920
-$Comp
-L Device:R_US R6
-U 1 1 5E651B8D
-P 3100 7340
-F 0 "R6" H 3168 7386 50  0000 L CNN
-F 1 "100" H 3168 7295 50  0000 L CNN
-F 2 "" V 3140 7330 50  0001 C CNN
-F 3 "~" H 3100 7340 50  0001 C CNN
-	1    3100 7340
-	1    0    0    -1
-$EndComp
 Wire Wire Line
 	2800 6920 2800 7190
@@
 Text Notes 3780 790  0    197  ~ 39
 *
+$Comp
+L Switch:SW_SPST SW1
+U 1 1 5E660D37
+P 1470 1110
+F 0 "SW1" H 1470 1030 50  0000 C CNN
+F 1 "SW_SPST" H 1470 1254 50  0001 C CNN
+F 2 "Payload:GW12RCH" H 1470 1110 50  0001 C CNN
+F 3 "~" H 1470 1110 50  0001 C CNN
+	1    1470 1110
+	1    0    0    -1
+$EndComp
+Wire Wire Line
+	1040 1110 1270 1110
+Wire Wire Line
+	1670 1110 1730 1110
+Connection ~ 1730 1110
+$Comp
+L Device:R_US R3
+U 1 1 5E623A5D
+P 1580 7310
+F 0 "R3" H 1648 7356 50  0000 L CNN
+F 1 "100" H 1648 7265 50  0000 L CNN
+F 2 "Resistor_SMD:R_0805_2012Metric_Pad1.15x1.40mm_HandSolder" V 1620 7300 50  0001 C CNN
+F 3 "~" H 1580 7310 50  0001 C CNN
+	1    1580 7310
+	1    0    0    -1
+$EndComp
+$Comp
+L Device:R_US R6
+U 1 1 5E651B8D
+P 3100 7340
+F 0 "R6" H 3168 7386 50  0000 L CNN
+F 1 "100" H 3168 7295 50  0000 L CNN
+F 2 "Resistor_SMD:R_0805_2012Metric_Pad1.15x1.40mm_HandSolder" V 3140 7330 50  0001 C CNN
+F 3 "~" H 3100 7340 50  0001 C CNN
+	1    3100 7340
+	1    0    0    -1
+$EndComp
 $EndSCHEMATC

Commit message: Began routing Board B Adjusted board bridge to 10 pins to transfer both 3.3v rails
Parts:
- J2: footprint Connector_JST:JST_SH_BM09B-SRSS-TB_1x09-1MP_P1.00mm_Vertical -> Connector_JST:JST_SH_BM10B-SRSS-TB_1x10-1MP_P1.00mm_Vertical; symbol Connector_Generic:Conn_01x09 -> Connector_Generic:Conn_01x10
Connections:
- wire segments 103 -> 104
Changed lines of the file:
@@
 EESchema Schematic File Version 4
-LIBS:Payload2020A-cache
-EELAYER 29 0
+EELAYER 30 0
 EELAYER END
 $Descr A4 11693 8268
@@
 	8350 3820 8880 3820
 $Comp
-L Connector_Generic:Conn_01x09 J2
+L Connector_Generic:Conn_01x10 J2
 U 1 1 5E53BD04
 P 9730 2150
 F 0 "J2" H 9780 2767 50  0000 C CNN
 F 1 "BridgeConn" H 9780 2676 50  0000 C CNN
-F 2 "Connector_JST:JST_SH_BM09B-SRSS-TB_1x09-1MP_P1.00mm_Vertical" H 9730 2150 50  0001 C CNN
+F 2 "Connector_JST:JST_SH_BM10B-SRSS-TB_1x10-1MP_P1.00mm_Vertical" H 9730 2150 50  0001 C CNN
 F 3 "~" H 9730 2150 50  0001 C CNN
 	1    9730 2150
@@
 	1    0    0    -1
 $EndComp
+$Comp
+L power:+3V3 #PWR0101
+U 1 1 5E670EE5
+P 8870 2650
+F 0 "#PWR0101" H 8870 2500 50  0001 C CNN
+F 1 "+3V3" H 8885 2823 50  0000 C CNN
+F 2 "" H 8870 2650 50  0001 C CNN
+F 3 "" H 8870 2650 50  0001 C CNN
+	1    8870 2650
+	-1   0    0    -1
+$EndComp
+Wire Wire Line
+	8870 2650 9530 2650
 $EndSCHEMATC

Commit message: -Added corner mounting holes to each board -Added mounting holes for HX711 -CHECK HOLE SIZING TO MATCH 4-40
Parts:
- added H1, H2, H3, H4: Corner, MountingHole:MountingHole_3.2mm_M3, symbol Mechanical:MountingHole
- added H5, H6: HX711, MountingHole:MountingHole_3.2mm_M3, symbol Mechanical:MountingHole
Changed lines of the file:
@@
 EESchema Schematic File Version 4
-EELAYER 30 0
+LIBS:Payload2020A-cache
+EELAYER 29 0
 EELAYER END
 $Descr A4 11693 8268
@@
 Wire Wire Line
 	8870 2650 9530 2650
+$Comp
+L Mechanical:MountingHole H2
+U 1 1 5E69D126
+P 4370 7650
+F 0 "H2" H 4470 7696 50  0000 L CNN
+F 1 "Corner" H 4470 7605 50  0000 L CNN
+F 2 "MountingHole:MountingHole_3.2mm_M3" H 4370 7650 50  0001 C CNN
+F 3 "~" H 4370 7650 50  0001 C CNN
+	1    4370 7650
+	1    0    0    -1
+$EndComp
+$Comp
+L Mechanical:MountingHole H1
+U 1 1 5E69D7F4
+P 4370 7420
+F 0 "H1" H 4470 7466 50  0000 L CNN
+F 1 "Corner" H 4470 7375 50  0000 L CNN
+F 2 "MountingHole:MountingHole_3.2mm_M3" H 4370 7420 50  0001 C CNN
+F 3 "~" H 4370 7420 50  0001 C CNN
+	1    4370 7420
+	1    0    0    -1
+$EndComp
+$Comp
+L Mechanical:MountingHole H4
+U 1 1 5E6A359E
+P 4830 7650
+F 0 "H4" H 4930 7696 50  0000 L CNN
+F 1 "Corner" H 4930 7605 50  0000 L CNN
+F 2 "MountingHole:MountingHole_3.2mm_M3" H 4830 7650 50  0001 C CNN
+F 3 "~" H 4830 7650 50  0001 C CNN
+	1    4830 7650
+	1    0    0    -1
+$EndComp
+$Comp
+L Mechanical:MountingHole H3
+U 1 1 5E6A35A4
+P 4830 7420
+F 0 "H3" H 4930 7466 50  0000 L CNN
+F 1 "Corner" H 4930 7375 50  0000 L CNN
+F 2 "MountingHole:MountingHole_3.2mm_M3" H 4830 7420 50  0001 C CNN
+F 3 "~" H 4830 7420 50  0001 C CNN
+	1    4830 7420
+	1    0    0    -1
+$EndComp
+$Comp
+L Mechanical:MountingHole H5
+U 1 1 5E6B8F67
+P 5410 7420
+F 0 "H5" H 5510 7466 50  0000 L CNN
+F 1 "HX711" H 5510 7375 50  0000 L CNN
+F 2 "MountingHole:MountingHole_3.2mm_M3" H 5410 7420 50  0001 C CNN
+F 3 "~" H 5410 7420 50  0001 C CNN
+	1    5410 7420
+	1    0    0    -1
+$EndComp
+$Comp
+L Mechanical:MountingHole H6
+U 1 1 5E6B9A49
+P 5410 7650
+F 0 "H6" H 5510 7696 50  0000 L CNN
+F 1 "HX711" H 5510 7605 50  0000 L CNN
+F 2 "MountingHole:MountingHole_3.2mm_M3" H 5410 7650 50  0001 C CNN
+F 3 "~" H 5410 7650 50  0001 C CNN
+	1    5410 7650
+	1    0    0    -1
+$EndComp
 $EndSCHEMATC

Commit message: Created 4-40 thread mounting hole Selected 4-40 hole size for Board A
Parts:
- H1, H2, H3, H4: footprint MountingHole:MountingHole_3.2mm_M3 -> Payload2020:MountingHole_4-40
Changed lines of the file:
@@
 EESchema Schematic File Version 4
-LIBS:Payload2020A-cache
-EELAYER 29 0
+EELAYER 30 0
 EELAYER END
 $Descr A4 11693 8268
@@
 F 0 "H2" H 4470 7696 50  0000 L CNN
 F 1 "Corner" H 4470 7605 50  0000 L CNN
-F 2 "MountingHole:MountingHole_3.2mm_M3" H 4370 7650 50  0001 C CNN
+F 2 "Payload2020:MountingHole_4-40" H 4370 7650 50  0001 C CNN
 F 3 "~" H 4370 7650 50  0001 C CNN
 	1    4370 7650
@@
 F 0 "H1" H 4470 7466 50  0000 L CNN
 F 1 "Corner" H 4470 7375 50  0000 L CNN
-F 2 "MountingHole:MountingHole_3.2mm_M3" H 4370 7420 50  0001 C CNN
+F 2 "Payload2020:MountingHole_4-40" H 4370 7420 50  0001 C CNN
 F 3 "~" H 4370 7420 50  0001 C CNN
 	1    4370 7420
@@
 F 0 "H4" H 4930 7696 50  0000 L CNN
 F 1 "Corner" H 4930 7605 50  0000 L CNN
-F 2 "MountingHole:MountingHole_3.2mm_M3" H 4830 7650 50  0001 C CNN
+F 2 "Payload2020:MountingHole_4-40" H 4830 7650 50  0001 C CNN
 F 3 "~" H 4830 7650 50  0001 C CNN
 	1    4830 7650
@@
 F 0 "H3" H 4930 7466 50  0000 L CNN
 F 1 "Corner" H 4930 7375 50  0000 L CNN
-F 2 "MountingHole:MountingHole_3.2mm_M3" H 4830 7420 50  0001 C CNN
+F 2 "Payload2020:MountingHole_4-40" H 4830 7420 50  0001 C CNN
 F 3 "~" H 4830 7420 50  0001 C CNN
 	1    4830 7420

Commit message: Placed corner mounting holes on each board Drew backside ground plane on Board B
Parts:
- H1, H2, H3, H4: footprint Payload2020:MountingHole_4-40 -> Payload:MountingHole_4-40
Changed lines of the file:
@@
 EESchema Schematic File Version 4
-EELAYER 30 0
+LIBS:Payload2020A-cache
+EELAYER 29 0
 EELAYER END
 $Descr A4 11693 8268
@@
 F 0 "H2" H 4470 7696 50  0000 L CNN
 F 1 "Corner" H 4470 7605 50  0000 L CNN
-F 2 "Payload2020:MountingHole_4-40" H 4370 7650 50  0001 C CNN
+F 2 "Payload:MountingHole_4-40" H 4370 7650 50  0001 C CNN
 F 3 "~" H 4370 7650 50  0001 C CNN
 	1    4370 7650
@@
 F 0 "H1" H 4470 7466 50  0000 L CNN
 F 1 "Corner" H 4470 7375 50  0000 L CNN
-F 2 "Payload2020:MountingHole_4-40" H 4370 7420 50  0001 C CNN
+F 2 "Payload:MountingHole_4-40" H 4370 7420 50  0001 C CNN
 F 3 "~" H 4370 7420 50  0001 C CNN
 	1    4370 7420
@@
 F 0 "H4" H 4930 7696 50  0000 L CNN
 F 1 "Corner" H 4930 7605 50  0000 L CNN
-F 2 "Payload2020:MountingHole_4-40" H 4830 7650 50  0001 C CNN
+F 2 "Payload:MountingHole_4-40" H 4830 7650 50  0001 C CNN
 F 3 "~" H 4830 7650 50  0001 C CNN
 	1    4830 7650
@@
 F 0 "H3" H 4930 7466 50  0000 L CNN
 F 1 "Corner" H 4930 7375 50  0000 L CNN
-F 2 "Payload2020:MountingHole_4-40" H 4830 7420 50  0001 C CNN
+F 2 "Payload:MountingHole_4-40" H 4830 7420 50  0001 C CNN
 F 3 "~" H 4830 7420 50  0001 C CNN
 	1    4830 7420

Commit message: Checked and fixed alignment of HX711 footprint dimensions Added hx711 mounting hole directly to footprint Redrawn edge cuts to fit into payload bay with about 0.01" fudge factor
Parts:
- removed H5, H6: HX711, MountingHole:MountingHole_3.2mm_M3, symbol Mechanical:MountingHole
Changed lines of the file:
@@
-	1    0    0    -1
-$EndComp
-$Comp
-L Mechanical:MountingHole H5
-U 1 1 5E6B8F67
-P 5410 7420
-F 0 "H5" H 5510 7466 50  0000 L CNN
-F 1 "HX711" H 5510 7375 50  0000 L CNN
-F 2 "MountingHole:MountingHole_3.2mm_M3" H 5410 7420 50  0001 C CNN
-F 3 "~" H 5410 7420 50  0001 C CNN
-	1    5410 7420
-	1    0    0    -1
-$EndComp
-$Comp
-L Mechanical:MountingHole H6
-U 1 1 5E6B9A49
-P 5410 7650
-F 0 "H6" H 5510 7696 50  0000 L CNN
-F 1 "HX711" H 5510 7605 50  0000 L CNN
-F 2 "MountingHole:MountingHole_3.2mm_M3" H 5410 7650 50  0001 C CNN
-F 3 "~" H 5410 7650 50  0001 C CNN
-	1    5410 7650
 	1    0    0    -1
 $EndComp
