File: PCB files/PayloadBoard/Payload2020/Payload2020A.sch (KiCad schematic (older format))
At the start: 28 parts, among them J1 BATTERY, J2 BridgeConn, J3 LoadCell, Q1 Q_NMOS_GSD, Q2 Q_NMOS_GSD, SW1 SW_SPST, U1 Teensy3.6, U2 ArduCam, U3 HX711_Breakout, U4 AP7370-50W5-7, U5 TPS613222ADBVR

Commit message: Redrawn edge cuts for board B Redrawn GND planes Changed bridge connector to molex picoblade
Parts:
- J2: footprint Connector_JST:JST_SH_BM10B-SRSS-TB_1x10-1MP_P1.00mm_Vertical -> Connector_Molex:Molex_PicoBlade_53047-1010_1x10_P1.25mm_Vertical
Changed lines of the file:
@@
 F 0 "J2" H 9780 2767 50  0000 C CNN
 F 1 "BridgeConn" H 9780 2676 50  0000 C CNN
-F 2 "Connector_JST:JST_SH_BM10B-SRSS-TB_1x10-1MP_P1.00mm_Vertical" H 9730 2150 50  0001 C CNN
+F 2 "Connector_Molex:Molex_PicoBlade_53047-1010_1x10_P1.25mm_Vertical" H 9730 2150 50  0001 C CNN
 F 3 "~" H 9730 2150 50  0001 C CNN
 	1    9730 2150

Commit message: BIG changus -Fully routed both boards -Changed board to board connector to JST SH -Changed load cell connector to molex picoblade -Added silkscreen version & signature -Moved arducam connector to align with payload structure
Parts:
- J2: footprint Connector_Molex:Molex_PicoBlade_53047-1010_1x10_P1.25mm_Vertical -> Connector_JST:JST_SH_SM15B-SRSS-TB_1x15-1MP_P1.00mm_Horizontal; symbol Connector_Generic:Conn_01x10 -> Connector_Generic:Conn_01x15
- J3: footprint Connector_JST:JST_SH_BM04B-SRSS-TB_1x04-1MP_P1.00mm_Vertical -> Connector_Molex:Molex_PicoBlade_53047-0410_1x04_P1.25mm_Vertical
Connections:
- net labels added: DEN_G, DRDY_G, INT1_XM, INT2_XM, INT_G
- wire segments 104 -> 114
Changed lines of the file:
@@
 	8350 3820 8880 3820
 $Comp
-L Connector_Generic:Conn_01x10 J2
+L Connector_Generic:Conn_01x15 J2
 U 1 1 5E53BD04
-P 9730 2150
-F 0 "J2" H 9780 2767 50  0000 C CNN
-F 1 "BridgeConn" H 9780 2676 50  0000 C CNN
-F 2 "Connector_Molex:Molex_PicoBlade_53047-1010_1x10_P1.25mm_Vertical" H 9730 2150 50  0001 C CNN
-F 3 "~" H 9730 2150 50  0001 C CNN
-	1    9730 2150
-	1    0    0    -1
-$EndComp
-Text Label 9080 1750 0    50   ~ 0
+P 9420 2030
+F 0 "J2" H 9430 2930 50  0000 C CNN
+F 1 "BridgeConn" H 9430 2850 50  0000 C CNN
+F 2 "Connector_JST:JST_SH_SM15B-SRSS-TB_1x15-1MP_P1.00mm_Horizontal" H 9420 2030 50  0001 C CNN
+F 3 "~" H 9420 2030 50  0001 C CNN
+	1    9420 2030
+	1    0    0    -1
+$EndComp
+Text Label 8770 1330 0    50   ~ 0
 Berry_SDA
-Text Label 9080 1850 0    50   ~ 0
+Text Label 8770 1430 0    50   ~ 0
 Berry_SCL
 Text Label 7730 6220 2    50   ~ 0
@@
 L power:+3.3VA #PWR020
 U 1 1 5E5BD94E
-P 8870 2150
-F 0 "#PWR020" H 8870 2000 50  0001 C CNN
-F 1 "+3.3VA" H 8885 2323 50  0000 C CNN
-F 2 "" H 8870 2150 50  0001 C CNN
-F 3 "" H 8870 2150 50  0001 C CNN
-	1    8870 2150
-	1    0    0    -1
-$EndComp
-Wire Wire Line
-	9530 2150 8870 2150
+P 8560 1730
+F 0 "#PWR020" H 8560 1580 50  0001 C CNN
+F 1 "+3.3VA" H 8575 1903 50  0000 C CNN
+F 2 "" H 8560 1730 50  0001 C CNN
+F 3 "" H 8560 1730 50  0001 C CNN
+	1    8560 1730
+	1    0    0    -1
+$EndComp
+Wire Wire Line
+	9220 1730 8560 1730
 Wire Wire Line
 	1040 1210 1150 1210
@@
 Wire Wire Line
 	3240 1460 3240 1400
-Text Label 9080 2450 0    50   ~ 0
+Text Label 8770 2030 0    50   ~ 0
 XBEE_DOUT
-Text Label 9080 2550 0    50   ~ 0
+Text Label 8770 2130 0    50   ~ 0
 XBEE_DIN
 Wire Wire Line
-	9080 1750 9530 1750
-Wire Wire Line
-	9080 1850 9530 1850
-Wire Wire Line
-	9080 2350 9530 2350
-Wire Wire Line
-	9080 2450 9530 2450
-Wire Wire Line
-	9080 2550 9530 2550
-Wire Wire Line
-	9080 1950 9530 1950
-Text Label 9080 1950 0    50   ~ 0
+	8770 1330 9220 1330
+Wire Wire Line
+	8770 1430 9220 1430
+Wire Wire Line
+	8770 1930 9220 1930
+Wire Wire Line
+	8770 2030 9220 2030
+Wire Wire Line
+	8770 2130 9220 2130
+Wire Wire Line
+	8770 1530 9220 1530
+Text Label 8770 1530 0    50   ~ 0
 RX_GPS
 Wire Wire Line
-	9080 2050 9530 2050
-Text Label 9080 2050 0    50   ~ 0
+	8770 1630 9220 1630
+Text Label 8770 1630 0    50   ~ 0
 TX_GPS
 Wire Wire Line
-	9080 2250 9530 2250
-Text Label 9080 2350 0    50   ~ 0
+	8770 1830 9220 1830
+Text Label 8770 1930 0    50   ~ 0
 XBEE_CTS
-Text Label 9080 2250 0    50   ~ 0
+Text Label 8770 1830 0    50   ~ 0
 XBEE_RTS
 Text Label 4630 3920 0    50   ~ 0
@@
 F 0 "J3" H 10032 3695 50  0000 C CNN
 F 1 "LoadCell" H 10032 3786 50  0000 C CNN
-F 2 "Connector_JST:JST_SH_BM04B-SRSS-TB_1x04-1MP_P1.00mm_Vertical" H 10140 4120 50  0001 C CNN
+F 2 "Connector_Molex:Molex_PicoBlade_53047-0410_1x04_P1.25mm_Vertical" H 10140 4120 50  0001 C CNN
 F 3 "~" H 10140 4120 50  0001 C CNN
 	1    10140 4120
@@
 L power:+3V3 #PWR0101
 U 1 1 5E670EE5
-P 8870 2650
-F 0 "#PWR0101" H 8870 2500 50  0001 C CNN
-F 1 "+3V3" H 8885 2823 50  0000 C CNN
-F 2 "" H 8870 2650 50  0001 C CNN
-F 3 "" H 8870 2650 50  0001 C CNN
-	1    8870 2650
+P 8560 2230
+F 0 "#PWR0101" H 8560 2080 50  0001 C CNN
+F 1 "+3V3" H 8575 2403 50  0000 C CNN
+F 2 "" H 8560 2230 50  0001 C CNN
+F 3 "" H 8560 2230 50  0001 C CNN
+	1    8560 2230
 	-1   0    0    -1
 $EndComp
 Wire Wire Line
-	8870 2650 9530 2650
+	8560 2230 9220 2230
 $Comp
 L Mechanical:MountingHole H2
@@
 	1    0    0    -1
 $EndComp
+Text Label 8770 2330 0    50   ~ 0
+DEN_G
+Text Label 8770 2430 0    50   ~ 0
+INT_G
+Text Label 8770 2530 0    50   ~ 0
+DRDY_G
+Text Label 8770 2630 0    50   ~ 0
+INT1_XM
+Text Label 8770 2730 0    50   ~ 0
+INT2_XM
+Wire Wire Line
+	8770 2330 9220 2330
+Wire Wire Line
+	8770 2430 9220 2430
+Wire Wire Line
+	9220 2530 8770 2530
+Wire Wire Line
+	8770 2630 9220 2630
+Wire Wire Line
+	8770 2730 9220 2730
+Text Label 4630 2620 0    50   ~ 0
+DEN_G
+Wire Wire Line
+	4630 2620 5080 2620
+Text Label 4630 2820 0    50   ~ 0
+INT_G
+Wire Wire Line
+	4630 2820 5080 2820
+Text Label 4630 2920 0    50   ~ 0
+DRDY_G
+Wire Wire Line
+	4630 2920 5080 2920
+Text Label 4630 3120 0    50   ~ 0
+INT1_XM
+Wire Wire Line
+	4630 3120 5080 3120
+Text Label 4630 3420 0    50   ~ 0
+INT2_XM
+Wire Wire Line
+	4630 3420 5080 3420
 $EndSCHEMATC
