File: PCB files/PayloadBoard/Payload2020/Payload2020B/Payload2020B.sch (KiCad schematic (older format))
At the start: 1 part

Commit message: -Created berryimuv3 symbol -Renamed Xbee symbol pins to match xbee pins on sparkfun explorer schematic, design now calls for xbee direct mount into PCB
Parts:
- added U?: BerryIMUv3, symbol PayloadBoard:BerryIMUv3
Changed lines of the file:
@@
 EESchema Schematic File Version 4
-EELAYER 30 0
+LIBS:Payload2020B-cache
+EELAYER 29 0
 EELAYER END
 $Descr A4 11693 8268
@@
 	1    0    0    -1
 $EndComp
+$Comp
+L PayloadBoard:BerryIMUv3 U?
+U 1 1 5E536455
+P 6770 3570
+F 0 "U?" H 6745 4285 50  0000 C CNN
+F 1 "BerryIMUv3" H 6745 4194 50  0000 C CNN
+F 2 "" H 6770 4270 50  0001 C CNN
+F 3 "" H 6770 4270 50  0001 C CNN
+	1    6770 3570
+	1    0    0    -1
+$EndComp

Commit message: -Added connector to Board B -Added descriptive i2c local net names
Parts:
- added J?: Conn_02x10_Counter_Clockwise, symbol Connector_Generic:Conn_02x10_Counter_Clockwise
Connections:
- net labels added: Berry_SCL, Berry_SDA
- wire segments 0 -> 4
Other:
- note removed: "change symbol pinout to match xbee module directly\n"
- moved on the sheet: U?
Changed lines of the file:
@@
 EESchema Schematic File Version 4
-LIBS:Payload2020B-cache
-EELAYER 29 0
+EELAYER 30 0
 EELAYER END
 $Descr A4 11693 8268
@@
 EndData
 $EndBitmap
-Text Notes 4100 2450 0    50   ~ 0
-change symbol pinout to match xbee module directly\n
 $Comp
 L PayloadBoard:Xbee_XBP9B U?
 U 1 1 5E49EA3B
-P 4300 3550
-F 0 "U?" H 4425 4225 50  0000 C CNN
-F 1 "Xbee_XBP9B" H 4425 4134 50  0000 C CNN
-F 2 "" H 3900 4100 50  0001 C CNN
-F 3 "" H 3900 4100 50  0001 C CNN
-	1    4300 3550
+P 5100 2200
+F 0 "U?" H 5225 2875 50  0000 C CNN
+F 1 "Xbee_XBP9B" H 5225 2784 50  0000 C CNN
+F 2 "" H 4700 2750 50  0001 C CNN
+F 3 "" H 4700 2750 50  0001 C CNN
+	1    5100 2200
 	1    0    0    -1
 $EndComp
@@
 L PayloadBoard:BerryIMUv3 U?
 U 1 1 5E536455
-P 6770 3570
-F 0 "U?" H 6745 4285 50  0000 C CNN
-F 1 "BerryIMUv3" H 6745 4194 50  0000 C CNN
-F 2 "" H 6770 4270 50  0001 C CNN
-F 3 "" H 6770 4270 50  0001 C CNN
-	1    6770 3570
+P 5350 4250
+F 0 "U?" H 5325 4965 50  0000 C CNN
+F 1 "BerryIMUv3" H 5325 4874 50  0000 C CNN
+F 2 "" H 5350 4950 50  0001 C CNN
+F 3 "" H 5350 4950 50  0001 C CNN
+	1    5350 4250
 	1    0    0    -1
 $EndComp
+$Comp
+L Connector_Generic:Conn_02x10_Counter_Clockwise J?
+U 1 1 5E544EC7
+P 7300 3200
+F 0 "J?" H 7350 3817 50  0000 C CNN
+F 1 "Conn_02x10_Counter_Clockwise" H 7350 3726 50  0000 C CNN
+F 2 "" H 7300 3200 50  0001 C CNN
+F 3 "~" H 7300 3200 50  0001 C CNN
+	1    7300 3200
+	1    0    0    -1
+$EndComp
+Text Label 4100 3900 0    50   ~ 0
+Berry_SDA
+Text Label 4100 4000 0    50   ~ 0
+Berry_SCL
+Wire Wire Line
+	4100 4000 4500 4000
+Wire Wire Line
+	4100 3900 4500 3900
+Text Label 6700 2800 0    50   ~ 0
+Berry_SDA
+Wire Wire Line
+	6700 2800 7100 2800
+Text Label 6700 2900 0    50   ~ 0
+Berry_SCL
+Wire Wire Line
+	6700 2900 7100 2900
 $EndSCHEMATC

Commit message: Payload Board B changes -Added xbee and berry GPS signal pin local nets -Added power and gnd flags to berry and xbee
Parts:
- J?: value Conn_02x10_Counter_Clockwise -> BridgeConn
Connections:
- net labels added: +3.3VA, +3V3, GNDREF, RX_GPS, XBEE_CTS, XBEE_DTR, XBEE_RTS
- wire segments 4 -> 16
Changed lines of the file:
@@
 EESchema Schematic File Version 4
-EELAYER 30 0
+LIBS:Payload2020B-cache
+EELAYER 29 0
 EELAYER END
 $Descr A4 11693 8268
@@
 P 7300 3200
 F 0 "J?" H 7350 3817 50  0000 C CNN
-F 1 "Conn_02x10_Counter_Clockwise" H 7350 3726 50  0000 C CNN
+F 1 "BridgeConn" H 7350 3726 50  0000 C CNN
 F 2 "" H 7300 3200 50  0001 C CNN
 F 3 "~" H 7300 3200 50  0001 C CNN
@@
 Wire Wire Line
 	6700 2900 7100 2900
+$Comp
+L power:+3.3VA #PWR?
+U 1 1 5E54854E
+P 4650 1700
+F 0 "#PWR?" H 4650 1550 50  0001 C CNN
+F 1 "+3.3VA" H 4665 1873 50  0000 C CNN
+F 2 "" H 4650 1700 50  0001 C CNN
+F 3 "" H 4650 1700 50  0001 C CNN
+	1    4650 1700
+	1    0    0    -1
+$EndComp
+Wire Wire Line
+	4650 1700 4650 1750
+$Comp
+L power:+3V3 #PWR?
+U 1 1 5E5493FD
+P 4500 3700
+F 0 "#PWR?" H 4500 3550 50  0001 C CNN
+F 1 "+3V3" H 4515 3873 50  0000 C CNN
+F 2 "" H 4500 3700 50  0001 C CNN
+F 3 "" H 4500 3700 50  0001 C CNN
+	1    4500 3700
+	1    0    0    -1
+$EndComp
+Wire Wire Line
+	4500 3700 4500 3800
+$Comp
+L power:GNDREF #PWR?
+U 1 1 5E54A258
+P 6800 3900
+F 0 "#PWR?" H 6800 3650 50  0001 C CNN
+F 1 "GNDREF" H 6805 3727 50  0000 C CNN
+F 2 "" H 6800 3900 50  0001 C CNN
+F 3 "" H 6800 3900 50  0001 C CNN
+	1    6800 3900
+	1    0    0    -1
+$EndComp
+Wire Wire Line
+	6800 3900 6150 3900
+Text Label 6450 4000 2    50   ~ 0
+RX_GPS
+Wire Wire Line
+	6450 4000 6150 4000
+Text Label 6700 3000 0    50   ~ 0
+RX_GPS
+Wire Wire Line
+	6700 3000 7100 3000
+$Comp
+L power:GNDREF #PWR?
+U 1 1 5E54D3B7
+P 4650 2690
+F 0 "#PWR?" H 4650 2440 50  0001 C CNN
+F 1 "GNDREF" H 4655 2517 50  0000 C CNN
+F 2 "" H 4650 2690 50  0001 C CNN
+F 3 "" H 4650 2690 50  0001 C CNN
+	1    4650 2690
+	1    0    0    -1
+$EndComp
+Wire Wire Line
+	4650 2690 4650 2650
+Text Label 6220 2150 2    50   ~ 0
+XBEE_RTS
+Text Label 6220 2550 2    50   ~ 0
+XBEE_CTS
+Wire Wire Line
+	5800 2150 6220 2150
+Wire Wire Line
+	6220 2550 5800 2550
+Text Label 4230 2550 0    50   ~ 0
+XBEE_DTR
+Wire Wire Line
+	4230 2550 4650 2550
+Text Label 6700 3100 0    50   ~ 0
+XBEE_RTS
+Text Label 6700 3200 0    50   ~ 0
+XBEE_CTS
+Text Label 6700 3300 0    50   ~ 0
+XBEE_DTR
+Wire Wire Line
+	6700 3100 7100 3100
+Wire Wire Line
+	7100 3200 6700 3200
+Wire Wire Line
+	6700 3300 7100 3300
 $EndSCHEMATC

Commit message: -Fixed xbee serial nets -Berrygps nets now include tx/rx for gps
Connections:
- net labels added: TX_GPS, XBEE_DIN, XBEE_DOUT
- net labels removed: XBEE_DTR
- wire segments 16 -> 19
Other:
- note added: "Xbee\nSerial pins\nDOUT\nDIN\nCTS\nRTS"
- moved on the sheet: U?
Changed lines of the file:
@@
 L PayloadBoard:Xbee_XBP9B U?
 U 1 1 5E49EA3B
-P 5100 2200
-F 0 "U?" H 5225 2875 50  0000 C CNN
-F 1 "Xbee_XBP9B" H 5225 2784 50  0000 C CNN
-F 2 "" H 4700 2750 50  0001 C CNN
-F 3 "" H 4700 2750 50  0001 C CNN
-	1    5100 2200
+P 5100 2000
+F 0 "U?" H 5225 2675 50  0000 C CNN
+F 1 "Xbee_XBP9B" H 5225 2584 50  0000 C CNN
+F 2 "" H 4700 2550 50  0001 C CNN
+F 3 "" H 4700 2550 50  0001 C CNN
+	1    5100 2000
 	1    0    0    -1
 $EndComp
@@
 L Connector_Generic:Conn_02x10_Counter_Clockwise J?
 U 1 1 5E544EC7
-P 7300 3200
-F 0 "J?" H 7350 3817 50  0000 C CNN
-F 1 "BridgeConn" H 7350 3726 50  0000 C CNN
-F 2 "" H 7300 3200 50  0001 C CNN
-F 3 "~" H 7300 3200 50  0001 C CNN
-	1    7300 3200
+P 7700 3080
+F 0 "J?" H 7750 3697 50  0000 C CNN
+F 1 "BridgeConn" H 7750 3606 50  0000 C CNN
+F 2 "" H 7700 3080 50  0001 C CNN
+F 3 "~" H 7700 3080 50  0001 C CNN
+	1    7700 3080
 	1    0    0    -1
 $EndComp
@@
 Wire Wire Line
 	4100 3900 4500 3900
-Text Label 6700 2800 0    50   ~ 0
+Text Label 7070 2680 0    50   ~ 0
 Berry_SDA
 Wire Wire Line
-	6700 2800 7100 2800
-Text Label 6700 2900 0    50   ~ 0
+	7070 2680 7500 2680
+Text Label 7070 2780 0    50   ~ 0
 Berry_SCL
 Wire Wire Line
-	6700 2900 7100 2900
+	7070 2780 7500 2780
 $Comp
 L power:+3.3VA #PWR?
 U 1 1 5E54854E
-P 4650 1700
-F 0 "#PWR?" H 4650 1550 50  0001 C CNN
-F 1 "+3.3VA" H 4665 1873 50  0000 C CNN
-F 2 "" H 4650 1700 50  0001 C CNN
-F 3 "" H 4650 1700 50  0001 C CNN
-	1    4650 1700
+P 4650 1500
+F 0 "#PWR?" H 4650 1350 50  0001 C CNN
+F 1 "+3.3VA" H 4665 1673 50  0000 C CNN
+F 2 "" H 4650 1500 50  0001 C CNN
+F 3 "" H 4650 1500 50  0001 C CNN
+	1    4650 1500
 	1    0    0    -1
 $EndComp
 Wire Wire Line
-	4650 1700 4650 1750
+	4650 1500 4650 1550
 $Comp
 L power:+3V3 #PWR?
@@
 Wire Wire Line
 	6450 4000 6150 4000
-Text Label 6700 3000 0    50   ~ 0
+Text Label 7070 2880 0    50   ~ 0
 RX_GPS
 Wire Wire Line
-	6700 3000 7100 3000
+	7070 2880 7500 2880
 $Comp
 L power:GNDREF #PWR?
 U 1 1 5E54D3B7
-P 4650 2690
-F 0 "#PWR?" H 4650 2440 50  0001 C CNN
-F 1 "GNDREF" H 4655 2517 50  0000 C CNN
-F 2 "" H 4650 2690 50  0001 C CNN
-F 3 "" H 4650 2690 50  0001 C CNN
-	1    4650 2690
+P 4650 2490
+F 0 "#PWR?" H 4650 2240 50  0001 C CNN
+F 1 "GNDREF" H 4655 2317 50  0000 C CNN
+F 2 "" H 4650 2490 50  0001 C CNN
+F 3 "" H 4650 2490 50  0001 C CNN
+	1    4650 2490
 	1    0    0    -1
 $EndComp
 Wire Wire Line
-	4650 2690 4650 2650
-Text Label 6220 2150 2    50   ~ 0
+	4650 2490 4650 2450
+Text Label 6220 1950 2    50   ~ 0
 XBEE_RTS
-Text Label 6220 2550 2    50   ~ 0
+Text Label 6220 2350 2    50   ~ 0
 XBEE_CTS
 Wire Wire Line
-	5800 2150 6220 2150
+	5800 1950 6220 1950
 Wire Wire Line
-	6220 2550 5800 2550
-Text Label 4230 2550 0    50   ~ 0
-XBEE_DTR
+	6220 2350 5800 2350
+Text Label 7070 3080 0    50   ~ 0
+XBEE_RTS
+Text Label 7070 3180 0    50   ~ 0
+XBEE_CTS
 Wire Wire Line
-	4230 2550 4650 2550
-Text Label 6700 3100 0    50   ~ 0
-XBEE_RTS
-Text Label 6700 3200 0    50   ~ 0
-XBEE_CTS
-Text Label 6700 3300 0    50   ~ 0
-XBEE_DTR
+	7070 3080 7500 3080
 Wire Wire Line
-	6700 3100 7100 3100
+	7500 3180 7070 3180
+Text Label 4230 1750 0    50   ~ 0
+XBEE_DIN
+Text Label 4230 1650 0    50   ~ 0
+XBEE_DOUT
 Wire Wire Line
-	7100 3200 6700 3200
+	4230 1650 4650 1650
 Wire Wire Line
-	6700 3300 7100 3300
+	4650 1750 4230 1750
+Text Label 7070 3280 0    50   ~ 0
+XBEE_DOUT
+Text Label 7070 3380 0    50   ~ 0
+XBEE_DIN
+Wire Wire Line
+	7070 3380 7500 3380
+Wire Wire Line
+	7500 3280 7070 3280
+Text Notes 6460 2260 0    50   ~ 0
+Xbee\nSerial pins\nDOUT\nDIN\nCTS\nRTS
+Text Label 6450 4100 2    50   ~ 0
+TX_GPS
+Wire Wire Line
+	6450 4100 6150 4100
 $EndSCHEMATC

Commit message: Removed 5V regulator Stepped input voltage down to that of a 1s battery pack Added internal parallite battery connection
Other:
- note added: "Xbee Serial pins\nDOUT\nDIN\nCTS\nRTS"
- note removed: "Xbee\nSerial pins\nDOUT\nDIN\nCTS\nRTS"
Changed lines of the file:
@@
 	7500 3280 7070 3280
 Text Notes 6460 2260 0    50   ~ 0
-Xbee\nSerial pins\nDOUT\nDIN\nCTS\nRTS
+Xbee Serial pins\nDOUT\nDIN\nCTS\nRTS
 Text Label 6450 4100 2    50   ~ 0
 TX_GPS

Commit message: -began footprint for berryIMU -Added XBEE sparkfun footprints from github -Added xbee and gps net connection to connector on board A
Parts:
- J1: renamed from J?; symbol Connector_Generic:Conn_02x10_Counter_Clockwise -> Connector_Generic:Conn_01x09
- U1, U2: renamed from U?; footprint (none) -> SparkFunRF:XBEE-1
Connections:
- wire segments 19 -> 21
Changed lines of the file:
@@
 $EndBitmap
 $Comp
-L PayloadBoard:Xbee_XBP9B U?
+L PayloadBoard:Xbee_XBP9B U1
 U 1 1 5E49EA3B
 P 5100 2000
-F 0 "U?" H 5225 2675 50  0000 C CNN
+F 0 "U1" H 5225 2675 50  0000 C CNN
 F 1 "Xbee_XBP9B" H 5225 2584 50  0000 C CNN
-F 2 "" H 4700 2550 50  0001 C CNN
+F 2 "SparkFunRF:XBEE-1" H 4700 2550 50  0001 C CNN
 F 3 "" H 4700 2550 50  0001 C CNN
 	1    5100 2000
@@
 $EndComp
 $Comp
-L PayloadBoard:BerryIMUv3 U?
+L PayloadBoard:BerryIMUv3 U2
 U 1 1 5E536455
 P 5350 4250
-F 0 "U?" H 5325 4965 50  0000 C CNN
+F 0 "U2" H 5325 4965 50  0000 C CNN
 F 1 "BerryIMUv3" H 5325 4874 50  0000 C CNN
-F 2 "" H 5350 4950 50  0001 C CNN
+F 2 "SparkFunRF:XBEE-1" H 5350 4950 50  0001 C CNN
 F 3 "" H 5350 4950 50  0001 C CNN
 	1    5350 4250
@@
 $EndComp
 $Comp
-L Connector_Generic:Conn_02x10_Counter_Clockwise J?
+L Connector_Generic:Conn_01x09 J1
 U 1 1 5E544EC7
 P 7700 3080
-F 0 "J?" H 7750 3697 50  0000 C CNN
+F 0 "J1" H 7750 3697 50  0000 C CNN
 F 1 "BridgeConn" H 7750 3606 50  0000 C CNN
 F 2 "" H 7700 3080 50  0001 C CNN
@@
 	7070 2780 7500 2780
 $Comp
-L power:+3.3VA #PWR?
+L power:+3.3VA #PWR0101
 U 1 1 5E54854E
 P 4650 1500
-F 0 "#PWR?" H 4650 1350 50  0001 C CNN
+F 0 "#PWR0101" H 4650 1350 50  0001 C CNN
 F 1 "+3.3VA" H 4665 1673 50  0000 C CNN
 F 2 "" H 4650 1500 50  0001 C CNN
@@
 	4650 1500 4650 1550
 $Comp
-L power:+3V3 #PWR?
+L power:+3V3 #PWR0102
 U 1 1 5E5493FD
 P 4500 3700
-F 0 "#PWR?" H 4500 3550 50  0001 C CNN
+F 0 "#PWR0102" H 4500 3550 50  0001 C CNN
 F 1 "+3V3" H 4515 3873 50  0000 C CNN
 F 2 "" H 4500 3700 50  0001 C CNN
@@
 	4500 3700 4500 3800
 $Comp
-L power:GNDREF #PWR?
+L power:GNDREF #PWR0103
 U 1 1 5E54A258
 P 6800 3900
-F 0 "#PWR?" H 6800 3650 50  0001 C CNN
+F 0 "#PWR0103" H 6800 3650 50  0001 C CNN
 F 1 "GNDREF" H 6805 3727 50  0000 C CNN
 F 2 "" H 6800 3900 50  0001 C CNN
@@
 	7070 2880 7500 2880
 $Comp
-L power:GNDREF #PWR?
+L power:GNDREF #PWR0104
 U 1 1 5E54D3B7
 P 4650 2490
-F 0 "#PWR?" H 4650 2240 50  0001 C CNN
+F 0 "#PWR0104" H 4650 2240 50  0001 C CNN
 F 1 "GNDREF" H 4655 2317 50  0000 C CNN
 F 2 "" H 4650 2490 50  0001 C CNN
@@
 Wire Wire Line
 	6220 2350 5800 2350
-Text Label 7070 3080 0    50   ~ 0
-XBEE_RTS
-Text Label 7070 3180 0    50   ~ 0
+Text Label 7070 3280 0    50   ~ 0
 XBEE_CTS
 Wire Wire Line
-	7070 3080 7500 3080
-Wire Wire Line
-	7500 3180 7070 3180
+	7500 3280 7070 3280
 Text Label 4230 1750 0    50   ~ 0
 XBEE_DIN
@@
 Wire Wire Line
 	4650 1750 4230 1750
-Text Label 7070 3280 0    50   ~ 0
+Text Label 7070 3380 0    50   ~ 0
 XBEE_DOUT
-Text Label 7070 3380 0    50   ~ 0
+Text Label 7070 3480 0    50   ~ 0
 XBEE_DIN
 Wire Wire Line
-	7070 3380 7500 3380
+	7070 3480 7500 3480
 Wire Wire Line
-	7500 3280 7070 3280
+	7500 3380 7070 3380
 Text Notes 6460 2260 0    50   ~ 0
 Xbee Serial pins\nDOUT\nDIN\nCTS\nRTS
@@
 Wire Wire Line
 	6450 4100 6150 4100
+$Comp
+L power:+3.3VA #PWR0105
+U 1 1 5E5F28CD
+P 6910 3080
+F 0 "#PWR0105" H 6910 2930 50  0001 C CNN
+F 1 "+3.3VA" H 6925 3253 50  0000 C CNN
+F 2 "" H 6910 3080 50  0001 C CNN
+F 3 "" H 6910 3080 50  0001 C CNN
+	1    6910 3080
+	1    0    0    -1
+$EndComp
+Wire Wire Line
+	6910 3080 7500 3080
+Wire Wire Line
+	7070 3180 7500 3180
+Text Label 7070 3180 0    50   ~ 0
+XBEE_RTS
+Text Label 7070 2980 0    50   ~ 0
+TX_GPS
+Wire Wire Line
+	7070 2980 7500 2980
 $EndSCHEMATC

Commit message: Arranged more components on board -Drew board edges for board B -Added User controlled LEDs
Parts:
- J1: footprint (none) -> Connector_JST:JST_EH_S9B-EH_1x09_P2.50mm_Horizontal
- U2: footprint SparkFunRF:XBEE-1 -> Payload:BerryGPS-IMU_V3
Changed lines of the file:
@@
 F 0 "U2" H 5325 4965 50  0000 C CNN
 F 1 "BerryIMUv3" H 5325 4874 50  0000 C CNN
-F 2 "SparkFunRF:XBEE-1" H 5350 4950 50  0001 C CNN
+F 2 "Payload:BerryGPS-IMU_V3" H 5350 4950 50  0001 C CNN
 F 3 "" H 5350 4950 50  0001 C CNN
 	1    5350 4250
@@
 F 0 "J1" H 7750 3697 50  0000 C CNN
 F 1 "BridgeConn" H 7750 3606 50  0000 C CNN
-F 2 "" H 7700 3080 50  0001 C CNN
+F 2 "Connector_JST:JST_EH_S9B-EH_1x09_P2.50mm_Horizontal" H 7700 3080 50  0001 C CNN
 F 3 "~" H 7700 3080 50  0001 C CNN
 	1    7700 3080

Commit message: -Selected all footprints -Began routing Board A
Parts:
- J1: footprint Connector_JST:JST_EH_S9B-EH_1x09_P2.50mm_Horizontal -> Connector_JST:JST_SH_BM09B-SRSS-TB_1x09-1MP_P1.00mm_Vertical
Connections:
- no-connect marks 0 -> 2
Other:
- moved on the sheet: U1
Changed lines of the file:
@@
 L PayloadBoard:Xbee_XBP9B U1
 U 1 1 5E49EA3B
-P 5100 2000
-F 0 "U1" H 5225 2675 50  0000 C CNN
-F 1 "Xbee_XBP9B" H 5225 2584 50  0000 C CNN
-F 2 "SparkFunRF:XBEE-1" H 4700 2550 50  0001 C CNN
-F 3 "" H 4700 2550 50  0001 C CNN
-	1    5100 2000
+P 5150 2600
+F 0 "U1" H 5275 3275 50  0000 C CNN
+F 1 "Xbee_XBP9B" H 5275 3184 50  0000 C CNN
+F 2 "SparkFunRF:XBEE-1" H 4750 3150 50  0001 C CNN
+F 3 "" H 4750 3150 50  0001 C CNN
+	1    5150 2600
 	1    0    0    -1
 $EndComp
@@
 L PayloadBoard:BerryIMUv3 U2
 U 1 1 5E536455
-P 5350 4250
-F 0 "U2" H 5325 4965 50  0000 C CNN
-F 1 "BerryIMUv3" H 5325 4874 50  0000 C CNN
-F 2 "Payload:BerryGPS-IMU_V3" H 5350 4950 50  0001 C CNN
-F 3 "" H 5350 4950 50  0001 C CNN
-	1    5350 4250
+P 5400 4850
+F 0 "U2" H 5375 5565 50  0000 C CNN
+F 1 "BerryIMUv3" H 5375 5474 50  0000 C CNN
+F 2 "Payload:BerryGPS-IMU_V3" H 5400 5550 50  0001 C CNN
+F 3 "" H 5400 5550 50  0001 C CNN
+	1    5400 4850
 	1    0    0    -1
 $EndComp
@@
 L Connector_Generic:Conn_01x09 J1
 U 1 1 5E544EC7
-P 7700 3080
-F 0 "J1" H 7750 3697 50  0000 C CNN
-F 1 "BridgeConn" H 7750 3606 50  0000 C CNN
-F 2 "Connector_JST:JST_EH_S9B-EH_1x09_P2.50mm_Horizontal" H 7700 3080 50  0001 C CNN
-F 3 "~" H 7700 3080 50  0001 C CNN
-	1    7700 3080
+P 7750 3680
+F 0 "J1" H 7800 4297 50  0000 C CNN
+F 1 "BridgeConn" H 7800 4206 50  0000 C CNN
+F 2 "Connector_JST:JST_SH_BM09B-SRSS-TB_1x09-1MP_P1.00mm_Vertical" H 7750 3680 50  0001 C CNN
+F 3 "~" H 7750 3680 50  0001 C CNN
+	1    7750 3680
 	1    0    0    -1
 $EndComp
-Text Label 4100 3900 0    50   ~ 0
+Text Label 4150 4500 0    50   ~ 0
 Berry_SDA
-Text Label 4100 4000 0    50   ~ 0
+Text Label 4150 4600 0    50   ~ 0
 Berry_SCL
 Wire Wire Line
-	4100 4000 4500 4000
+	4150 4600 4550 4600
 Wire Wire Line
-	4100 3900 4500 3900
-Text Label 7070 2680 0    50   ~ 0
+	4150 4500 4550 4500
+Text Label 7120 3280 0    50   ~ 0
 Berry_SDA
 Wire Wire Line
-	7070 2680 7500 2680
-Text Label 7070 2780 0    50   ~ 0
+	7120 3280 7550 3280
+Text Label 7120 3380 0    50   ~ 0
 Berry_SCL
 Wire Wire Line
-	7070 2780 7500 2780
+	7120 3380 7550 3380
 $Comp
 L power:+3.3VA #PWR0101
 U 1 1 5E54854E
-P 4650 1500
-F 0 "#PWR0101" H 4650 1350 50  0001 C CNN
-F 1 "+3.3VA" H 4665 1673 50  0000 C CNN
-F 2 "" H 4650 1500 50  0001 C CNN
-F 3 "" H 4650 1500 50  0001 C CNN
-	1    4650 1500
+P 4700 2100
+F 0 "#PWR0101" H 4700 1950 50  0001 C CNN
+F 1 "+3.3VA" H 4715 2273 50  0000 C CNN
+F 2 "" H 4700 2100 50  0001 C CNN
+F 3 "" H 4700 2100 50  0001 C CNN
+	1    4700 2100
 	1    0    0    -1
 $EndComp
 Wire Wire Line
-	4650 1500 4650 1550
+	4700 2100 4700 2150
 $Comp
 L power:+3V3 #PWR0102
 U 1 1 5E5493FD
-P 4500 3700
-F 0 "#PWR0102" H 4500 3550 50  0001 C CNN
-F 1 "+3V3" H 4515 3873 50  0000 C CNN
-F 2 "" H 4500 3700 50  0001 C CNN
-F 3 "" H 4500 3700 50  0001 C CNN
-	1    4500 3700
+P 4550 4300
+F 0 "#PWR0102" H 4550 4150 50  0001 C CNN
+F 1 "+3V3" H 4565 4473 50  0000 C CNN
+F 2 "" H 4550 4300 50  0001 C CNN
+F 3 "" H 4550 4300 50  0001 C CNN
+	1    4550 4300
 	1    0    0    -1
 $EndComp
 Wire Wire Line
-	4500 3700 4500 3800
+	4550 4300 4550 4400
 $Comp
 L power:GNDREF #PWR0103
 U 1 1 5E54A258
-P 6800 3900
-F 0 "#PWR0103" H 6800 3650 50  0001 C CNN
-F 1 "GNDREF" H 6805 3727 50  0000 C CNN
-F 2 "" H 6800 3900 50  0001 C CNN
-F 3 "" H 6800 3900 50  0001 C CNN
-	1    6800 3900
+P 6720 4500
+F 0 "#PWR0103" H 6720 4250 50  0001 C CNN
+F 1 "GNDREF" H 6725 4327 50  0001 C CNN
+F 2 "" H 6720 4500 50  0001 C CNN
+F 3 "" H 6720 4500 50  0001 C CNN
+	1    6720 4500
 	1    0    0    -1
 $EndComp
 Wire Wire Line
-	6800 3900 6150 3900
-Text Label 6450 4000 2    50   ~ 0
+	6720 4500 6200 4500
+Text Label 6500 4600 2    50   ~ 0
 RX_GPS
 Wire Wire Line
-	6450 4000 6150 4000
-Text Label 7070 2880 0    50   ~ 0
+	6500 4600 6200 4600
+Text Label 7120 3480 0    50   ~ 0
 RX_GPS
 Wire Wire Line
-	7070 2880 7500 2880
+	7120 3480 7550 3480
 $Comp
 L power:GNDREF #PWR0104
 U 1 1 5E54D3B7
-P 4650 2490
-F 0 "#PWR0104" H 4650 2240 50  0001 C CNN
-F 1 "GNDREF" H 4655 2317 50  0000 C CNN
-F 2 "" H 4650 2490 50  0001 C CNN
-F 3 "" H 4650 2490 50  0001 C CNN
-	1    4650 2490
+P 4700 3090
+F 0 "#PWR0104" H 4700 2840 50  0001 C CNN
+F 1 "GNDREF" H 4705 2917 50  0000 C CNN
+F 2 "" H 4700 3090 50  0001 C CNN
+F 3 "" H 4700 3090 50  0001 C CNN
+	1    4700 3090
 	1    0    0    -1
 $EndComp
 Wire Wire Line
-	4650 2490 4650 2450
-Text Label 6220 1950 2    50   ~ 0
+	4700 3090 4700 3050
+Text Label 6270 2550 2    50   ~ 0
 XBEE_RTS
-Text Label 6220 2350 2    50   ~ 0
+Text Label 6270 2950 2    50   ~ 0
 XBEE_CTS
 Wire Wire Line
-	5800 1950 6220 1950
+	5850 2550 6270 2550
 Wire Wire Line
-	6220 2350 5800 2350
-Text Label 7070 3280 0    50   ~ 0
+	6270 2950 5850 2950
+Text Label 7120 3880 0    50   ~ 0
 XBEE_CTS
 Wire Wire Line
-	7500 3280 7070 3280
-Text Label 4230 1750 0    50   ~ 0
+	7550 3880 7120 3880
+Text Label 4280 2350 0    50   ~ 0
 XBEE_DIN
-Text Label 4230 1650 0    50   ~ 0
+Text Label 4280 2250 0    50   ~ 0
 XBEE_DOUT
 Wire Wire Line
-	4230 1650 4650 1650
+	4280 2250 4700 2250
 Wire Wire Line
-	4650 1750 4230 1750
-Text Label 7070 3380 0    50   ~ 0
+	4700 2350 4280 2350
+Text Label 7120 3980 0    50   ~ 0
 XBEE_DOUT
-Text Label 7070 3480 0    50   ~ 0
+Text Label 7120 4080 0    50   ~ 0
 XBEE_DIN
 Wire Wire Line
-	7070 3480 7500 3480
+	7120 4080 7550 4080
 Wire Wire Line
-	7500 3380 7070 3380
-Text Notes 6460 2260 0    50   ~ 0
+	7550 3980 7120 3980
+Text Notes 6510 2860 0    50   ~ 0
 Xbee Serial pins\nDOUT\nDIN\nCTS\nRTS
-Text Label 6450 4100 2    50   ~ 0
+Text Label 6500 4700 2    50   ~ 0
 TX_GPS
 Wire Wire Line
-	6450 4100 6150 4100
+	6500 4700 6200 4700
 $Comp
 L power:+3.3VA #PWR0105
 U 1 1 5E5F28CD
-P 6910 3080
-F 0 "#PWR0105" H 6910 2930 50  0001 C CNN
-F 1 "+3.3VA" H 6925 3253 50  0000 C CNN
-F 2 "" H 6910 3080 50  0001 C CNN
-F 3 "" H 6910 3080 50  0001 C CNN
-	1    6910 3080
+P 6960 3680
+F 0 "#PWR0105" H 6960 3530 50  0001 C CNN
+F 1 "+3.3VA" H 6975 3853 50  0000 C CNN
+F 2 "" H 6960 3680 50  0001 C CNN
+F 3 "" H 6960 3680 50  0001 C CNN
+	1    6960 3680
 	1    0    0    -1
 $EndComp
 Wire Wire Line
-	6910 3080 7500 3080
+	6960 3680 7550 3680
 Wire Wire Line
-	7070 3180 7500 3180
-Text Label 7070 3180 0    50   ~ 0
+	7120 3780 7550 3780
+Text Label 7120 3780 0    50   ~ 0
 XBEE_RTS
-Text Label 7070 2980 0    50   ~ 0
+Text Label 7120 3580 0    50   ~ 0
 TX_GPS
 Wire Wire Line
-	7070 2980 7500 2980
+	7120 3580 7550 3580
+NoConn ~ 6200 4400
+NoConn ~ 4550 4700
 $EndSCHEMATC
