File: PCB files/PayloadBoard/Payload2020/Payload2020B/Payload2020B.sch (KiCad schematic (older format))
At the start: 3 parts, among them J1 BridgeConn, U1 Xbee_XBP9B, U2 BerryIMUv3

Commit message: Began routing Board B Adjusted board bridge to 10 pins to transfer both 3.3v rails
Parts:
- J1: footprint Connector_JST:JST_SH_BM09B-SRSS-TB_1x09-1MP_P1.00mm_Vertical -> Connector_JST:JST_SH_BM10B-SRSS-TB_1x10-1MP_P1.00mm_Vertical; symbol Connector_Generic:Conn_01x09 -> Connector_Generic:Conn_01x10
Connections:
- wire segments 21 -> 23
Changed lines of the file:
@@
 EESchema Schematic File Version 4
-LIBS:Payload2020B-cache
-EELAYER 29 0
+EELAYER 30 0
 EELAYER END
 $Descr A4 11693 8268
@@
 $EndComp
 $Comp
-L Connector_Generic:Conn_01x09 J1
+L Connector_Generic:Conn_01x10 J1
 U 1 1 5E544EC7
 P 7750 3680
 F 0 "J1" H 7800 4297 50  0000 C CNN
 F 1 "BridgeConn" H 7800 4206 50  0000 C CNN
-F 2 "Connector_JST:JST_SH_BM09B-SRSS-TB_1x09-1MP_P1.00mm_Vertical" H 7750 3680 50  0001 C CNN
+F 2 "Connector_JST:JST_SH_BM10B-SRSS-TB_1x10-1MP_P1.00mm_Vertical" H 7750 3680 50  0001 C CNN
 F 3 "~" H 7750 3680 50  0001 C CNN
 	1    7750 3680
@@
 NoConn ~ 6200 4400
 NoConn ~ 4550 4700
+Wire Wire Line
+	7550 4180 6950 4180
+Wire Wire Line
+	6950 4180 6950 4170
+$Comp
+L power:+3V3 #PWR0106
+U 1 1 5E66C1CB
+P 6950 4170
+F 0 "#PWR0106" H 6950 4020 50  0001 C CNN
+F 1 "+3V3" H 6965 4343 50  0000 C CNN
+F 2 "" H 6950 4170 50  0001 C CNN
+F 3 "" H 6950 4170 50  0001 C CNN
+	1    6950 4170
+	1    0    0    -1
+$EndComp
 $EndSCHEMATC

Commit message: -Added corner mounting holes to each board -Added mounting holes for HX711 -CHECK HOLE SIZING TO MATCH 4-40
Parts:
- added H1, H2, H3, H4: Corner, symbol Mechanical:MountingHole
Changed lines of the file:
@@
 EESchema Schematic File Version 4
-EELAYER 30 0
+LIBS:Payload2020B-cache
+EELAYER 29 0
 EELAYER END
 $Descr A4 11693 8268
@@
 	1    0    0    -1
 $EndComp
+$Comp
+L Mechanical:MountingHole H1
+U 1 1 5E698CBA
+P 960 7030
+F 0 "H1" H 1060 7076 50  0000 L CNN
+F 1 "Corner" H 1060 6985 50  0000 L CNN
+F 2 "" H 960 7030 50  0001 C CNN
+F 3 "~" H 960 7030 50  0001 C CNN
+	1    960  7030
+	1    0    0    -1
+$EndComp
+$Comp
+L Mechanical:MountingHole H2
+U 1 1 5E699A8A
+P 960 7290
+F 0 "H2" H 1060 7336 50  0000 L CNN
+F 1 "Corner" H 1060 7245 50  0000 L CNN
+F 2 "" H 960 7290 50  0001 C CNN
+F 3 "~" H 960 7290 50  0001 C CNN
+	1    960  7290
+	1    0    0    -1
+$EndComp
+$Comp
+L Mechanical:MountingHole H3
+U 1 1 5E699E54
+P 1470 7020
+F 0 "H3" H 1570 7066 50  0000 L CNN
+F 1 "Corner" H 1570 6975 50  0000 L CNN
+F 2 "" H 1470 7020 50  0001 C CNN
+F 3 "~" H 1470 7020 50  0001 C CNN
+	1    1470 7020
+	1    0    0    -1
+$EndComp
+$Comp
+L Mechanical:MountingHole H4
+U 1 1 5E69A3B4
+P 1470 7290
+F 0 "H4" H 1570 7336 50  0000 L CNN
+F 1 "Corner" H 1570 7245 50  0000 L CNN
+F 2 "" H 1470 7290 50  0001 C CNN
+F 3 "~" H 1470 7290 50  0001 C CNN
+	1    1470 7290
+	1    0    0    -1
+$EndComp

Commit message: Placed corner mounting holes on each board Drew backside ground plane on Board B
Parts:
- H1, H2, H3, H4: footprint (none) -> Payload:MountingHole_4-40
Changed lines of the file:
@@
 F 0 "H1" H 1060 7076 50  0000 L CNN
 F 1 "Corner" H 1060 6985 50  0000 L CNN
-F 2 "" H 960 7030 50  0001 C CNN
+F 2 "Payload:MountingHole_4-40" H 960 7030 50  0001 C CNN
 F 3 "~" H 960 7030 50  0001 C CNN
 	1    960  7030
@@
 F 0 "H2" H 1060 7336 50  0000 L CNN
 F 1 "Corner" H 1060 7245 50  0000 L CNN
-F 2 "" H 960 7290 50  0001 C CNN
+F 2 "Payload:MountingHole_4-40" H 960 7290 50  0001 C CNN
 F 3 "~" H 960 7290 50  0001 C CNN
 	1    960  7290
@@
 F 0 "H3" H 1570 7066 50  0000 L CNN
 F 1 "Corner" H 1570 6975 50  0000 L CNN
-F 2 "" H 1470 7020 50  0001 C CNN
+F 2 "Payload:MountingHole_4-40" H 1470 7020 50  0001 C CNN
 F 3 "~" H 1470 7020 50  0001 C CNN
 	1    1470 7020
@@
 F 0 "H4" H 1570 7336 50  0000 L CNN
 F 1 "Corner" H 1570 7245 50  0000 L CNN
-F 2 "" H 1470 7290 50  0001 C CNN
+F 2 "Payload:MountingHole_4-40" H 1470 7290 50  0001 C CNN
 F 3 "~" H 1470 7290 50  0001 C CNN
 	1    1470 7290

Commit message: Redrawn edge cuts for board B Redrawn GND planes Changed bridge connector to molex picoblade
Parts:
- J1: footprint Connector_JST:JST_SH_BM10B-SRSS-TB_1x10-1MP_P1.00mm_Vertical -> Connector_Molex:Molex_PicoBlade_53047-1010_1x10_P1.25mm_Vertical
Changed lines of the file:
@@
 F 0 "J1" H 7800 4297 50  0000 C CNN
 F 1 "BridgeConn" H 7800 4206 50  0000 C CNN
-F 2 "Connector_JST:JST_SH_BM10B-SRSS-TB_1x10-1MP_P1.00mm_Vertical" H 7750 3680 50  0001 C CNN
+F 2 "Connector_Molex:Molex_PicoBlade_53047-1010_1x10_P1.25mm_Vertical" H 7750 3680 50  0001 C CNN
 F 3 "~" H 7750 3680 50  0001 C CNN
 	1    7750 3680

Commit message: BIG changus -Fully routed both boards -Changed board to board connector to JST SH -Changed load cell connector to molex picoblade -Added silkscreen version & signature -Moved arducam connector to align with payload structure
Parts:
- J1: footprint Connector_Molex:Molex_PicoBlade_53047-1010_1x10_P1.25mm_Vertical -> Connector_JST:JST_SH_SM15B-SRSS-TB_1x15-1MP_P1.00mm_Horizontal; symbol Connector_Generic:Conn_01x10 -> Connector_Generic:Conn_01x15
Connections:
- wire segments 23 -> 28
Changed lines of the file:
@@
 $EndComp
 $Comp
-L Connector_Generic:Conn_01x10 J1
+L Connector_Generic:Conn_01x15 J1
 U 1 1 5E544EC7
-P 7750 3680
-F 0 "J1" H 7800 4297 50  0000 C CNN
-F 1 "BridgeConn" H 7800 4206 50  0000 C CNN
-F 2 "Connector_Molex:Molex_PicoBlade_53047-1010_1x10_P1.25mm_Vertical" H 7750 3680 50  0001 C CNN
-F 3 "~" H 7750 3680 50  0001 C CNN
-	1    7750 3680
-	1    0    0    -1
-$EndComp
-Text Label 4150 4500 0    50   ~ 0
+P 7770 4500
+F 0 "J1" H 7780 5410 50  0000 C CNN
+F 1 "BridgeConn" H 7780 5330 50  0000 C CNN
+F 2 "Connector_JST:JST_SH_SM15B-SRSS-TB_1x15-1MP_P1.00mm_Horizontal" H 7770 4500 50  0001 C CNN
+F 3 "~" H 7770 4500 50  0001 C CNN
+	1    7770 4500
+	1    0    0    -1
+$EndComp
+Text Label 4500 4500 0    50   ~ 0
 Berry_SDA
-Text Label 4150 4600 0    50   ~ 0
+Text Label 4500 4600 0    50   ~ 0
 Berry_SCL
 Wire Wire Line
-	4150 4600 4550 4600
-Wire Wire Line
-	4150 4500 4550 4500
-Text Label 7120 3280 0    50   ~ 0
+	4500 4600 4900 4600
+Wire Wire Line
+	4500 4500 4900 4500
+Text Label 7140 3800 0    50   ~ 0
 Berry_SDA
 Wire Wire Line
-	7120 3280 7550 3280
-Text Label 7120 3380 0    50   ~ 0
+	7140 3800 7570 3800
+Text Label 7140 3900 0    50   ~ 0
 Berry_SCL
 Wire Wire Line
-	7120 3380 7550 3380
+	7140 3900 7570 3900
 $Comp
 L power:+3.3VA #PWR0101
@@
 L power:+3V3 #PWR0102
 U 1 1 5E5493FD
-P 4550 4300
-F 0 "#PWR0102" H 4550 4150 50  0001 C CNN
-F 1 "+3V3" H 4565 4473 50  0000 C CNN
-F 2 "" H 4550 4300 50  0001 C CNN
-F 3 "" H 4550 4300 50  0001 C CNN
-	1    4550 4300
-	1    0    0    -1
-$EndComp
-Wire Wire Line
-	4550 4300 4550 4400
+P 4900 4300
+F 0 "#PWR0102" H 4900 4150 50  0001 C CNN
+F 1 "+3V3" H 4915 4473 50  0000 C CNN
+F 2 "" H 4900 4300 50  0001 C CNN
+F 3 "" H 4900 4300 50  0001 C CNN
+	1    4900 4300
+	1    0    0    -1
+$EndComp
+Wire Wire Line
+	4900 4300 4900 4400
 $Comp
 L power:GNDREF #PWR0103
 U 1 1 5E54A258
-P 6720 4500
-F 0 "#PWR0103" H 6720 4250 50  0001 C CNN
-F 1 "GNDREF" H 6725 4327 50  0001 C CNN
-F 2 "" H 6720 4500 50  0001 C CNN
-F 3 "" H 6720 4500 50  0001 C CNN
-	1    6720 4500
-	1    0    0    -1
-$EndComp
-Wire Wire Line
-	6720 4500 6200 4500
-Text Label 6500 4600 2    50   ~ 0
+P 6370 4500
+F 0 "#PWR0103" H 6370 4250 50  0001 C CNN
+F 1 "GNDREF" H 6375 4327 50  0001 C CNN
+F 2 "" H 6370 4500 50  0001 C CNN
+F 3 "" H 6370 4500 50  0001 C CNN
+	1    6370 4500
+	1    0    0    -1
+$EndComp
+Wire Wire Line
+	6150 4600 5850 4600
+Text Label 7140 4000 0    50   ~ 0
 RX_GPS
 Wire Wire Line
-	6500 4600 6200 4600
-Text Label 7120 3480 0    50   ~ 0
-RX_GPS
-Wire Wire Line
-	7120 3480 7550 3480
+	7140 4000 7570 4000
 $Comp
 L power:GNDREF #PWR0104
@@
 Wire Wire Line
 	6270 2950 5850 2950
-Text Label 7120 3880 0    50   ~ 0
+Text Label 7140 4400 0    50   ~ 0
 XBEE_CTS
 Wire Wire Line
-	7550 3880 7120 3880
+	7570 4400 7140 4400
 Text Label 4280 2350 0    50   ~ 0
 XBEE_DIN
@@
 Wire Wire Line
 	4700 2350 4280 2350
-Text Label 7120 3980 0    50   ~ 0
+Text Label 7140 4500 0    50   ~ 0
 XBEE_DOUT
-Text Label 7120 4080 0    50   ~ 0
+Text Label 7140 4600 0    50   ~ 0
 XBEE_DIN
 Wire Wire Line
-	7120 4080 7550 4080
-Wire Wire Line
-	7550 3980 7120 3980
+	7140 4600 7570 4600
+Wire Wire Line
+	7570 4500 7140 4500
 Text Notes 6510 2860 0    50   ~ 0
 Xbee Serial pins\nDOUT\nDIN\nCTS\nRTS
-Text Label 6500 4700 2    50   ~ 0
+Text Label 6150 4700 2    50   ~ 0
 TX_GPS
 Wire Wire Line
-	6500 4700 6200 4700
+	6150 4700 5850 4700
 $Comp
 L power:+3.3VA #PWR0105
 U 1 1 5E5F28CD
-P 6960 3680
-F 0 "#PWR0105" H 6960 3530 50  0001 C CNN
-F 1 "+3.3VA" H 6975 3853 50  0000 C CNN
-F 2 "" H 6960 3680 50  0001 C CNN
-F 3 "" H 6960 3680 50  0001 C CNN
-	1    6960 3680
-	1    0    0    -1
-$EndComp
-Wire Wire Line
-	6960 3680 7550 3680
-Wire Wire Line
-	7120 3780 7550 3780
-Text Label 7120 3780 0    50   ~ 0
+P 6980 4200
+F 0 "#PWR0105" H 6980 4050 50  0001 C CNN
+F 1 "+3.3VA" H 6995 4373 50  0000 C CNN
+F 2 "" H 6980 4200 50  0001 C CNN
+F 3 "" H 6980 4200 50  0001 C CNN
+	1    6980 4200
+	1    0    0    -1
+$EndComp
+Wire Wire Line
+	6980 4200 7570 4200
+Wire Wire Line
+	7140 4300 7570 4300
+Text Label 7140 4300 0    50   ~ 0
 XBEE_RTS
-Text Label 7120 3580 0    50   ~ 0
+Text Label 7140 4100 0    50   ~ 0
 TX_GPS
 Wire Wire Line
-	7120 3580 7550 3580
-NoConn ~ 6200 4400
-NoConn ~ 4550 4700
-Wire Wire Line
-	7550 4180 6950 4180
-Wire Wire Line
-	6950 4180 6950 4170
+	7140 4100 7570 4100
+NoConn ~ 4900 4700
+Wire Wire Line
+	7570 4700 6970 4700
+Wire Wire Line
+	6970 4700 6970 4690
 $Comp
 L power:+3V3 #PWR0106
 U 1 1 5E66C1CB
-P 6950 4170
-F 0 "#PWR0106" H 6950 4020 50  0001 C CNN
-F 1 "+3V3" H 6965 4343 50  0000 C CNN
-F 2 "" H 6950 4170 50  0001 C CNN
-F 3 "" H 6950 4170 50  0001 C CNN
-	1    6950 4170
+P 6970 4690
+F 0 "#PWR0106" H 6970 4540 50  0001 C CNN
+F 1 "+3V3" H 6985 4863 50  0000 C CNN
+F 2 "" H 6970 4690 50  0001 C CNN
+F 3 "" H 6970 4690 50  0001 C CNN
+	1    6970 4690
 	1    0    0    -1
 $EndComp
@@
 	1    0    0    -1
 $EndComp
+NoConn ~ 5850 4400
+Text Label 6150 4600 2    50   ~ 0
+RX_GPS
+Wire Wire Line
+	6370 4500 5850 4500
+Wire Wire Line
+	5850 4800 7570 4800
+Wire Wire Line
+	5850 4900 7570 4900
+Wire Wire Line
+	5850 5000 7570 5000
+Wire Wire Line
+	5850 5100 7570 5100
+Wire Wire Line
+	5850 5200 7570 5200
 $EndSCHEMATC
